File: Hardware/Segment/daughterboard_2sheetbackup.sch (EAGLE design)
At the start: 162 parts, among them IC1 PBQ79656PAPTQ1, IC2 PBQ79656PAPTQ1, T1 PBHV8115X, 115, T2 PBHV8115X, 115, X1 5566-12, X2 5566-12, X3 5566-16, X4 5566-12, X5 5566-12, X6 5566-16

Commit message: Fixed second chip, replaced caps with 0603
Parts:
- removed COMH: 5566-2, con-molex:5566-2
- added CCB42, CCB43: 2.2nf, rcl:C-EUC0603
- added RVC13, RVC14, RVC33, RVC34: 49, rcl:R-US_R0603
- C1, CCB0, CCB1, CCB10, CCB11, CCB12, CCB13, CCB14, CCB15, CCB16, CCB17, CCB18, CCB19, CCB2, CCB20, CCB21, CCB22, CCB23, CCB24, CCB25, CCB3, CCB4, CCB5, CCB6, CCB7, CCB8, CCB9, CVC0, CVC1, CVC2, CVC3, CVC4, CVC5, CVC6, CVC7, CVC8, CVC9: device rcl:C-EUC0603 -> capacitor-wima:C2.5/2
Connections:
- removed net COMHN: CCB50.1, COMH-1.S
- removed net COMHP: CCB49.1, COMH-2.S
- removed net N$125 (its old number): CCB45.2, IC2.COMLN, RVC32.2, RVC35.1
- removed net N$132 (its old number): CCB51.2, IC2.COMHN, RVC37.2, RVC39.2
- new net N$127: CCB45.2, IC2.COMHP, RVC32.2, RVC35.1
- new net N$128: CCB42.2, RVC31.1
- new net N$129: CCB43.2, RVC32.1
- new net N$130: CCB42.1, RVC33.2
- new net N$133: CCB48.2, IC2.COMLN, RVC37.1, RVC38.2
- new net N$134: CCB51.2, IC2.COMLP, RVC37.2, RVC39.2
- new net N$63: CCB16.1, RVC13.2
- new net N$64: CCB17.1, RVC14.2
- new net N$66: CCB25.1
- new net N$69: CCB24.1
- net COMLN: now also CCB49.1; no longer CCB24.1
- net COMLP: now also CCB50.1; no longer CCB25.1
- net COMMN: now also RVC33.1; no longer CCB16.1, RVC32.1
- net COMMP: now also RVC34.1; no longer CCB17.1, RVC31.1
- net N$126: now also IC2.COMHN; no longer IC2.COMLP
- net N$131: now also CCB43.1, RVC34.2; no longer CCB48.2, IC2.COMHP, RVC37.1, RVC38.2
