File: Hardware/Segment/daughterboard.sch (EAGLE design)
At the start: 175 parts, among them IC1 PBQ79656PAPTQ1, IC2 PBQ79656PAPTQ1, T1 PBHV8115X, 115, T2 PBHV8115X, 115

Commit message: Daughterboard fixes V2.1
Parts:
- removed GND, RX, TX: (no value), wirepad:2,54/1,0
- added UART: 22-23-2031, con-molex:22-23-2031
Connections:
- net GNDL: now also UART-3.S; no longer GND.P
- net N$3: now also UART-2.S; no longer RX.P
- net N$9: now also UART-1.S; no longer TX.P
Changed lines of the file:
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@@
 <part name="GNDL" library="wirepad" library_urn="urn:adsk.eagle:library:412" deviceset="SMD5" device="" package3d_urn="urn:adsk.eagle:package:30841/1"/>
 <part name="GNDH" library="wirepad" library_urn="urn:adsk.eagle:library:412" deviceset="SMD5" device="" package3d_urn="urn:adsk.eagle:package:30841/1"/>
-<part name="TX" library="wirepad" library_urn="urn:adsk.eagle:library:412" deviceset="2,54/1,0" device="" package3d_urn="urn:adsk.eagle:package:30828/1"/>
-<part name="RX" library="wirepad" library_urn="urn:adsk.eagle:library:412" deviceset="2,54/1,0" device="" package3d_urn="urn:adsk.eagle:package:30828/1"/>
-<part name="GND" library="wirepad" library_urn="urn:adsk.eagle:library:412" deviceset="2,54/1,0" device="" package3d_urn="urn:adsk.eagle:package:30828/1"/>
 <part name="NFAULT" library="testpad" library_urn="urn:adsk.eagle:library:385" deviceset="TP" device="B2,54" package3d_urn="urn:adsk.eagle:package:27948/1"/>
 <part name="RCS1" library="rcl" library_urn="urn:adsk.eagle:library:334" deviceset="R-US_" device="R0603" package3d_urn="urn:adsk.eagle:package:23555/3" value="10"/>
@@
 <part name="CCB10" library="rcl" library_urn="urn:adsk.eagle:library:334" deviceset="C-EU" device="C0603" package3d_urn="urn:adsk.eagle:package:23616/2" value="0.47uf"/>
 <part name="CCB10-1" library="rcl" library_urn="urn:adsk.eagle:library:334" deviceset="C-EU" device="C0603" package3d_urn="urn:adsk.eagle:package:23616/2" value="0.47uf"/>
+<part name="UART" library="con-molex" library_urn="urn:adsk.eagle:library:165" deviceset="22-23-2031" device="" package3d_urn="urn:adsk.eagle:package:8078634/1"/>
 </parts>
 <sheets>
@@
 <attribute name="VALUE" x="145.923" y="270.002" size="1.778" layer="96" rot="R180"/>
 </instance>
-<instance part="TX" gate="P" x="195.58" y="45.72" smashed="yes" rot="R180">
-<attribute name="NAME" x="196.723" y="43.8658" size="1.778" layer="95" rot="R180"/>
-<attribute name="VALUE" x="196.723" y="49.022" size="1.778" layer="96" rot="R180"/>
-</instance>
-<instance part="RX" gate="P" x="195.58" y="43.18" smashed="yes" rot="R180">
-<attribute name="NAME" x="196.723" y="41.3258" size="1.778" layer="95" rot="R180"/>
-<attribute name="VALUE" x="196.723" y="46.482" size="1.778" layer="96" rot="R180"/>
-</instance>
-<instance part="GND" gate="P" x="195.58" y="17.78" smashed="yes" rot="R90">
-<attribute name="NAME" x="193.7258" y="16.637" size="1.778" layer="95" rot="R90"/>
-<attribute name="VALUE" x="198.882" y="16.637" size="1.778" layer="96" rot="R90"/>
-</instance>
 <instance part="NFAULT" gate="G$1" x="193.04" y="68.58" smashed="yes" rot="R270">
 <attribute name="NAME" x="194.31" y="69.85" size="1.778" layer="95" rot="R270"/>
@@
 <attribute name="NAME" x="136.779" y="339.344" size="1.778" layer="95" rot="R90"/>
 <attribute name="VALUE" x="141.859" y="339.344" size="1.778" layer="96" rot="R90"/>
+</instance>
+<instance part="UART" gate="-1" x="195.58" y="45.72" smashed="yes">
+<attribute name="NAME" x="198.12" y="44.958" size="1.524" layer="95"/>
+<attribute name="VALUE" x="194.818" y="47.117" size="1.778" layer="96"/>
+</instance>
+<instance part="UART" gate="-2" x="195.58" y="43.18" smashed="yes">
+<attribute name="NAME" x="198.12" y="42.418" size="1.524" layer="95"/>
+</instance>
+<instance part="UART" gate="-3" x="200.66" y="25.4" smashed="yes">
+<attribute name="NAME" x="203.2" y="24.638" size="1.524" layer="95"/>
 </instance>
 </instances>
@@
 <pinref part="CDVDD" gate="G$1" pin="1"/>
 <wire x1="198.12" y1="38.1" x2="198.12" y2="35.56" width="0.1524" layer="91"/>
-<wire x1="198.12" y1="35.56" x2="198.12" y2="20.32" width="0.1524" layer="91"/>
-<wire x1="198.12" y1="20.32" x2="195.58" y2="20.32" width="0.1524" layer="91"/>
+<wire x1="198.12" y1="35.56" x2="198.12" y2="25.4" width="0.1524" layer="91"/>
 <junction x="198.12" y="35.56"/>
 <junction x="172.72" y="20.32"/>
 <pinref part="IC1" gate="G$1" pin="AVSS?"/>
-<wire x1="195.58" y1="20.32" x2="175.26" y2="20.32" width="0.1524" layer="91"/>
+<wire x1="198.12" y1="25.4" x2="198.12" y2="20.32" width="0.1524" layer="91"/>
+<wire x1="198.12" y1="20.32" x2="175.26" y2="20.32" width="0.1524" layer="91"/>
 <wire x1="175.26" y1="20.32" x2="172.72" y2="20.32" width="0.1524" layer="91"/>
 <wire x1="190.5" y1="76.2" x2="198.12" y2="76.2" width="0.1524" layer="91"/>
@@
 <pinref part="GNDL" gate="1" pin="P"/>
 <junction x="149.86" y="17.78"/>
-<pinref part="GND" gate="P" pin="P"/>
-<junction x="195.58" y="20.32"/>
+<pinref part="UART" gate="-3" pin="S"/>
+<junction x="198.12" y="25.4"/>
 </segment>
 <segment>
@@
 <wire x1="180.34" y1="43.18" x2="190.5" y2="43.18" width="0.1524" layer="91"/>
 <wire x1="193.04" y1="43.18" x2="190.5" y2="43.18" width="0.1524" layer="91"/>
-<pinref part="RX" gate="P" pin="P"/>
 <junction x="190.5" y="43.18"/>
+<pinref part="UART" gate="-2" pin="S"/>
 </segment>
 </net>
@@
 <pinref part="IC1" gate="G$1" pin="TX"/>
 <wire x1="193.04" y1="45.72" x2="190.5" y2="45.72" width="0.1524" layer="91"/>
-<pinref part="TX" gate="P" pin="P"/>
-</segment>
-</net>
+<pinref part="UART" gate="-1" pin="S"/>
+</segment>
+</net>

Commit message: Added two-color LEDs to BMS daughterboard to indicate balancing current status and direction
Parts:
- added LED1, LED10, LED11, LED12, LED13, LED14, LED15, LED16, LED17, LED18, LED19, LED2, LED20, LED21, LED22, LED3, LED4, LED5, LED6, LED7, LED8, LED9: APHB1608SGEC, APHB1608SGEC:APHB1608SGEC
- added R1, R10, R11, R12, R13, R14, R15, R16, R17, R18, R19, R2, R20, R21, R22, R3, R4, R5, R6, R7, R8, R9: 150, rcl:R-US_R0603
Connections:
- net N$19 renamed VC1-IN
- net N$20 renamed VC2-IN
- net N$22 renamed VC3-IN
- net N$23 renamed VC4-IN
- net N$24 renamed VC9-IN
- net N$25 renamed VC8-IN
- net N$26 renamed VC7-IN
- net N$28 renamed VC6-IN
- net N$30 renamed VC5-IN
- net N$34 renamed VC9-IN-1
- net N$35 renamed VC8-IN-1
- net N$36 renamed VC7-IN-1
- net N$37 renamed VC6-IN-1
- net N$38 renamed VC5-IN-1
- net N$39 renamed VC4-IN-1
- net N$40 renamed VC3-IN-1
- net N$41 renamed VC2-IN-1
- net N$42 renamed VC1-IN-1
- removed net N$32: CBL-1.S, RCB0.1
- removed net N$72: CBH-3.S, RCB2-1.1
- removed net N$73: CBH-2.S, RCB1-1.1
- removed net N$75: CBH-4.S, RCB3-1.1
- removed net N$78: CBH-5.S, RCB4-1.1
- removed net N$81: CBH-6.S, RCB5-1.1
- removed net N$84: CBH-7.S, RCB6-1.1
- removed net N$87: CBH-8.S, RCB7-1.1
- removed net N$90: CBH-9.S, RCB8-1.1
- removed net N$93: CBH-10.S, RCB9-1.1
- removed net N$96: CBH-1.S, RCB0-1.1
- new net CB0-IN: CBL-1.S, LED1.A_GREEN, LED1.K_RED, RCB0.1
- new net CB0-IN-1: CBH-1.S, LED12.A_GREEN, LED12.K_RED, RCB0-1.1
- new net CB1-IN: CBL-2.S, LED2.A_GREEN, LED2.K_RED, RCB1.1
- new net CB1-IN-1: CBH-2.S, LED13.A_GREEN, LED13.K_RED, RCB1-1.1
- new net CB10-IN: CBL-11.S, LED11.A_GREEN, LED11.K_RED, RCB10.1
- new net CB10-IN-1: CBH-11.S, LED22.A_GREEN, LED22.K_RED, RCB10-1.1
- new net CB2-IN: CBL-3.S, LED3.A_GREEN, LED3.K_RED, RCB2.1
- new net CB2-IN-1: CBH-3.S, LED14.A_GREEN, LED14.K_RED, RCB2-1.1
- new net CB3-IN: CBL-4.S, LED4.A_GREEN, LED4.K_RED, RCB3.1
- new net CB3-IN-1: CBH-4.S, LED15.A_GREEN, LED15.K_RED, RCB3-1.1
- new net CB4-IN: CBL-5.S, LED5.A_GREEN, LED5.K_RED, RCB4.1
- new net CB4-IN-1: CBH-5.S, LED16.A_GREEN, LED16.K_RED, RCB4-1.1
- new net CB5-IN: CBL-6.S, LED6.A_GREEN, LED6.K_RED, RCB5.1
- new net CB5-IN-1: CBH-6.S, LED17.A_GREEN, LED17.K_RED, RCB5-1.1
- new net CB6-IN: CBL-7.S, LED7.A_GREEN, LED7.K_RED, RCB6.1
- new net CB6-IN-1: CBH-7.S, LED18.A_GREEN, LED18.K_RED, RCB6-1.1
- new net CB7-IN: CBL-8.S, LED8.A_GREEN, LED8.K_RED, RCB7.1
- new net CB7-IN-1: CBH-8.S, LED19.A_GREEN, LED19.K_RED, RCB7-1.1
- new net CB8-IN: CBL-9.S, LED9.A_GREEN, LED9.K_RED, RCB8.1
- new net CB8-IN-1: CBH-9.S, LED20.A_GREEN, LED20.K_RED, RCB8-1.1
- new net CB9-IN: CBL-10.S, LED10.A_GREEN, LED10.K_RED, RCB9.1
- new net CB9-IN-1: CBH-10.S, LED21.A_GREEN, LED21.K_RED, RCB9-1.1
- new net N$14: LED15.A_RED, LED15.K_GREEN, R15.1
- new net N$19: LED18.A_RED, LED18.K_GREEN, R18.1
- new net N$20: LED19.A_RED, LED19.K_GREEN, R19.1
- new net N$22: LED20.A_RED, LED20.K_GREEN, R20.1
- new net N$23: LED21.A_RED, LED21.K_GREEN, R21.1
- new net N$24: LED6.A_RED, LED6.K_GREEN, R6.1
- new net N$25: LED22.A_RED, LED22.K_GREEN, R22.1
- new net N$35: LED9.A_RED, LED9.K_GREEN, R9.1
- new net N$38: LED10.A_RED, LED10.K_GREEN, R10.1
- new net N$41: LED11.A_RED, LED11.K_GREEN, R11.1
- new net N$43: LED1.A_RED, LED1.K_GREEN, R1.1
- net CB0: now also R1.2
- net CB0-1: now also R12.2
- net CB1: now also R2.2
- net CB1-1: now also R13.2
- net CB10: now also R11.2
- net CB10-1: now also R22.2
- net CB2: now also R3.2
- net CB2-1: now also R14.2
- net CB3: now also R4.2
- net CB3-1: now also R15.2
- net CB4: now also R5.2
- net CB4-1: now also R16.2
- net CB5: now also R6.2
- net CB5-1: now also R17.2
- net CB6: now also R7.2
- net CB6-1: now also R18.2
- net CB7: now also R8.2
- net CB7-1: now also R19.2
- net CB8: now also R9.2
- net CB8-1: now also R20.2
- net CB9: now also R10.2
- net CB9-1: now also R21.2
- net N$11: now also LED14.A_RED, LED14.K_GREEN, R14.1; no longer CBL-11.S, RCB10.1
- net N$12: now also LED3.A_RED, LED3.K_GREEN, R3.1; no longer CBL-5.S, RCB4.1
- net N$15: now also LED16.A_RED, LED16.K_GREEN, R16.1; no longer CBL-6.S, RCB5.1
- net N$17: now also LED17.A_RED, LED17.K_GREEN, R17.1; no longer CBH-11.S, RCB10-1.1
- net N$18: now also LED4.A_RED, LED4.K_GREEN, R4.1; no longer CBL-9.S, RCB8.1
- net N$21: now also LED5.A_RED, LED5.K_GREEN, R5.1; no longer CBL-10.S, RCB9.1
- net N$27: now also LED7.A_RED, LED7.K_GREEN, R7.1; no longer CBL-7.S, RCB6.1
- net N$31: now also LED8.A_RED, LED8.K_GREEN, R8.1; no longer CBL-8.S, RCB7.1
- net N$5: now also LED12.A_RED, LED12.K_GREEN, R12.1; no longer CBL-2.S, RCB1.1
- net N$6: now also LED2.A_RED, LED2.K_GREEN, R2.1; no longer CBL-3.S, RCB2.1
- net N$8: now also LED13.A_RED, LED13.K_GREEN, R13.1; no longer CBL-4.S, RCB3.1

Commit message: BMS V3 hardware
Parts:
- removed CBH, CBL, VCH: 5566-12, con-molex:5566-12
- removed TEMPH, TEMPL: 5566-16, con-molex:5566-16
- added J1, J2: DF11-16DP-2DSA(01), hirose_connectors:DF11-16DP-2DSA(01)
- added VCL1, VCL2, VCL3: DF11-12DP-2DSA(01), hirose_connectors:DF11-12DP-2DSA(01)
- COMH, COML, SR: value 5566-2 -> DF11-4DP-2DSA(24); device con-molex:5566-2 -> hirose_connectors:DF11-4DP-2DSA(24)
- VCL: value 5566-12 -> DF11-12DP-2DSA(01); device con-molex:5566-12 -> hirose_connectors:DF11-12DP-2DSA(01)
Connections:
- net BATC: now also VCL.11; no longer VCL-11.S
- net BATC-1: now also VCL2.11; no longer VCH-11.S
- net CB0-IN: now also VCL1.1; no longer CBL-1.S
- net CB0-IN-1: now also VCL3.1; no longer CBH-1.S
- net CB1-IN: now also VCL1.2; no longer CBL-2.S
- net CB1-IN-1: now also VCL3.2; no longer CBH-2.S
- net CB10-IN: now also VCL1.11; no longer CBL-11.S
- net CB10-IN-1: now also VCL3.11; no longer CBH-11.S
- net CB2-IN: now also VCL1.3; no longer CBL-3.S
- net CB2-IN-1: now also VCL3.3; no longer CBH-3.S
- net CB3-IN: now also VCL1.4; no longer CBL-4.S
- net CB3-IN-1: now also VCL3.4; no longer CBH-4.S
- net CB4-IN: now also VCL1.5; no longer CBL-5.S
- net CB4-IN-1: now also VCL3.5; no longer CBH-5.S
- net CB5-IN: now also VCL1.6; no longer CBL-6.S
- net CB5-IN-1: now also VCL3.6; no longer CBH-6.S
- net CB6-IN: now also VCL1.7; no longer CBL-7.S
- net CB6-IN-1: now also VCL3.7; no longer CBH-7.S
- net CB7-IN: now also VCL1.8; no longer CBL-8.S
- net CB7-IN-1: now also VCL3.8; no longer CBH-8.S
- net CB8-IN: now also VCL1.9; no longer CBL-9.S
- net CB8-IN-1: now also VCL3.9; no longer CBH-9.S
- net CB9-IN: now also VCL1.10; no longer CBL-10.S
- net CB9-IN-1: now also VCL3.10; no longer CBH-10.S
- net COMHN: now also COMH.4; no longer COMH-1.S
- net COMHP: now also COMH.3; no longer COMH-2.S
- net COMLN: now also COML.1; no longer COML-1.S
- net COMLP: now also COML.2; no longer COML-2.S
- net GNDH: now also J2.10, J2.12, J2.14, J2.16, J2.2, J2.4, J2.6, J2.8, VCL2.1; no longer TEMPH-10.S, TEMPH-11.S, TEMPH-12.S, TEMPH-13.S, TEMPH-14.S, TEMPH-15.S, TEMPH-16.S, TEMPH-9.S, VCH-1.S
- net GNDL: now also J1.10, J1.12, J1.14, J1.16, J1.2, J1.4, J1.6, J1.8, VCL.1; no longer TEMPL-10.S, TEMPL-11.S, TEMPL-12.S, TEMPL-13.S, TEMPL-14.S, TEMPL-15.S, TEMPL-16.S, TEMPL-9.S, VCL-1.S
- net N$13: now also RCS1.1, SR.1; no longer RCS2.1, SR-2.S
- net N$16: now also RCS2.1, SR.4; no longer RCS1.1, SR-1.S
- net TEMP1: now also J1.1; no longer TEMPL-1.S
- net TEMP10: now also J2.3; no longer TEMPH-2.S
- net TEMP11: now also J2.5; no longer TEMPH-3.S
- net TEMP12: now also J2.7; no longer TEMPH-4.S
- net TEMP13: now also J2.9; no longer TEMPH-5.S
- net TEMP14: now also J2.11; no longer TEMPH-6.S
- net TEMP15: now also J2.13; no longer TEMPH-7.S
- net TEMP16: now also J2.15; no longer TEMPH-8.S
- net TEMP2: now also J1.3; no longer TEMPL-2.S
- net TEMP3: now also J1.5; no longer TEMPL-3.S
- net TEMP4: now also J1.7; no longer TEMPL-4.S
- net TEMP5: now also J1.9; no longer TEMPL-5.S
- net TEMP6: now also J1.11; no longer TEMPL-6.S
- net TEMP7: now also J1.13; no longer TEMPL-7.S
- net TEMP8: now also J1.15; no longer TEMPL-8.S
- net TEMP9: now also J2.1; no longer TEMPH-1.S
- net VC1-IN: now also VCL.2; no longer VCL-2.S
- net VC1-IN-1: now also VCL2.2; no longer VCH-2.S
- net VC2-IN: now also VCL.3; no longer VCL-3.S
- net VC2-IN-1: now also VCL2.3; no longer VCH-3.S
- net VC3-IN: now also VCL.4; no longer VCL-4.S
- net VC3-IN-1: now also VCL2.4; no longer VCH-4.S
- net VC4-IN: now also VCL.5; no longer VCL-5.S
- net VC4-IN-1: now also VCL2.5; no longer VCH-5.S
- net VC5-IN: now also VCL.6; no longer VCL-6.S
- net VC5-IN-1: now also VCL2.6; no longer VCH-6.S
- net VC6-IN: now also VCL.7; no longer VCL-7.S
- net VC6-IN-1: now also VCL2.7; no longer VCH-7.S
- net VC7-IN: now also VCL.8; no longer VCL-8.S
- net VC7-IN-1: now also VCL2.8; no longer VCH-8.S
- net VC8-IN: now also VCL.9; no longer VCL-9.S
- net VC8-IN-1: now also VCL2.9; no longer VCH-9.S
- net VC9-IN: now also VCL.10; no longer VCL-10.S
- net VC9-IN-1: now also VCL2.10; no longer VCH-10.S
