File: Hardware/Segment - Copy/daughterboard.sch (EAGLE design)
At the start: 162 parts, among them IC1 PBQ79656PAPTQ1, IC2 PBQ79656PAPTQ1, T1 PBHV8115X, 115, T2 PBHV8115X, 115

Commit message: Daughterboard layout
Parts:
- renumbered RCOMH to CCOMH
Connections:
- net COMHN: now also COMH-1.S; no longer COMH-2.S
- net COMHP: now also COMH-2.S; no longer COMH-1.S
- net GND: now also CAVDD.1, CCOMMLN.2, CCOMMLP.1, CCVDD.1, CDVDD.1, CNEG5V.1, CREFHP.1, IC1.AVSS, IC1.AVSS?, IC1.CVSS, IC1.DVSS, IC1.REFHM
- net GND-1: now also CAVDD-1.1, CCOMMHN.1, CCOMMHP.2, CCVDD-1.1, CDVDD-1.1, CNEG5V-1.1, CREFHP-1.1, IC2.AVSS, IC2.AVSS?, IC2.CVSS, IC2.DVSS, IC2.REFHM
- net GNDN: no longer CAVDD.1, CCOMMLN.2, CCOMMLP.1, CCVDD.1, CDVDD.1, CNEG5V.1, CREFHP.1, IC1.AVSS, IC1.AVSS?, IC1.CVSS, IC1.DVSS, IC1.REFHM
- net GNDN-1: no longer CAVDD-1.1, CCOMMHN.1, CCOMMHP.2, CCVDD-1.1, CDVDD-1.1, CNEG5V-1.1, CREFHP-1.1, IC2.AVSS, IC2.AVSS?, IC2.CVSS, IC2.DVSS, IC2.REFHM
- net N$131: now also CCOMH.1; no longer CCOMH.2
- net N$132: now also CCOMH.2; no longer CCOMH.1
Other:
- moved on the sheet: CAVDD-1, CCOMHN, CCOMHNG, CCOMHP, CCOMHPG, CCVDD-1, CDVDD-1, CNEG5V-1, CREFHP-1, RCOMHN, RCOMHP
