File: Hardware/Segment - Copy/daughterboard_2sheetbackup.sch (EAGLE design)
At the start: 162 parts, among them IC1 PBQ79656PAPTQ1, IC2 PBQ79656PAPTQ1, T1 PBHV8115X, 115, T2 PBHV8115X, 115

Commit message: Daughterboard layout
Parts:
- removed CAVDD, CAVDD-1, CDVDD, CDVDD-1, CREFHP, CREFHP-1: 1uf, rcl:C-EUC0603
- removed CBAT, CBAT-1: 10 nf, rcl:C-EUC0603
- removed CBH, VCH: 5566-12, con-molex:5566-12
- removed CCB0-1, CCB1-1, CCB2-1, CCB3-1, CCB4-1, CCB5-1, CCB6-1, CCB7-1, CCB8-1, CCB9-1, CVC0-1, CVC1-1, CVC2-1, CVC3-1, CVC4-1, CVC5-1, CVC6-1, CVC7-1, CVC8-1, CVC9-1: 0.47uf, rcl:C-EUC0603
- removed CCOMHN, CCOMHP, CCOMLN, CCOMLP, CCOMMN, CCOMMP: 2.2nf, rcl:C-EUC0603
- removed CCOMHNG, CCOMHPG, CCOMLNG, CCOMLPG: 220 pF, rcl:C-EUC0603
- removed CCOMMHN, CCOMMHP, CCOMMLN, CCOMMLP: 220pf, rcl:C-EUC0603
- removed CCVDD, CCVDD-1: 4.7uf, rcl:C-EUC0603
- removed CNEG5V, CNEG5V-1, CNPN2, CNPN2-1: 0.1uf, rcl:C-EUC0603
- removed CNPN1, CNPN1-1: 0.22uf, rcl:C-EUC0603
- removed COMH: 5566-2, con-molex:5566-2
- removed CTSREF1, CTSREF2: 1 uF, rcl:C-EUC0603
- removed ESDCOMH: ESDAVLC6-2BLY, ESDAVLC6-2BLY:ESDAVLC6-2BLY
- removed RBAT-1: 30, rcl:R-US_R0603
- removed RCB0-1, RCB1-1, RCB10-1, RCB2-1, RCB3-1, RCB4-1, RCB5-1, RCB6-1, RCB7-1, RCB8-1, RCB9-1: 10, rcl:R-US_R1210
- removed RCOMH, RCOMMH: 1k, rcl:R-US_R0603
- removed RCOMHN, RCOMHP, RCOMMHN, RCOMMHP, RNPN-1: 49, rcl:R-US_R0603
- removed RVC0-1, RVC1-1, RVC10-1, RVC2-1, RVC3-1, RVC4-1, RVC5-1, RVC6-1, RVC7-1, RVC8-1, RVC9-1: 100, rcl:R-US_R0603
- removed TEMPH: 5566-16, con-molex:5566-16
- removed TEMPR10, TEMPR11, TEMPR12, TEMPR13, TEMPR14, TEMPR15, TEMPR16, TEMPR9: 10k, rcl:R-US_R0603
- added C1: 1 uF, capacitor-wima:C2.5/2
- added C2: 1 uF, rcl:C-EUC0603
- added CCB10: 10 nf, capacitor-wima:C2.5/2
- added CCB11, CCB12, CCB15: 1uf, capacitor-wima:C2.5/2
- added CCB13, CCB20: 0.1uf, capacitor-wima:C2.5/2
- added CCB14: 4.7uf, capacitor-wima:C2.5/2
- added CCB16, CCB17, CCB24, CCB25: 2.2nf, capacitor-wima:C2.5/2
- added CCB18, CCB19: 220pf, capacitor-wima:C2.5/2
- added CCB21: 0.22uf, capacitor-wima:C2.5/2
- added CCB22, CCB23: 220 pF, capacitor-wima:C2.5/2
- added CCB26, CCB27, CCB28, CCB29, CCB30, CCB31, CCB32, CCB33, CCB34, CCB35, CVC10, CVC11, CVC12, CVC13, CVC14, CVC15, CVC16, CVC17, CVC18, CVC19: 0.47uf, rcl:C-EUC0603
- added CCB36: 10 nf, rcl:C-EUC0603
- added CCB37, CCB38, CCB41: 1uf, rcl:C-EUC0603
- added CCB39, CCB46: 0.1uf, rcl:C-EUC0603
- added CCB40: 4.7uf, rcl:C-EUC0603
- added CCB42, CCB43, CCB49, CCB50: 2.2nf, rcl:C-EUC0603
- added CCB44, CCB45: 220pf, rcl:C-EUC0603
- added CCB47: 0.22uf, rcl:C-EUC0603
- added CCB48, CCB51: 220 pF, rcl:C-EUC0603
- added D2: ESDAVLC6-2BLY, ESDAVLC6-2BLY:ESDAVLC6-2BLY
- added R10, R11, R12, R13, R14, R15, R16, R9: 10k, rcl:R-US_R0603
- added RCB12, RCB13, RCB14, RCB15, RCB16, RCB17, RCB18, RCB19, RCB20, RCB21, RCB22: 10, rcl:R-US_R0603
- added RCB23: 30, rcl:R-US_R0603
- added RVC13, RVC14, RVC31, RVC32, RVC33, RVC34, RVC36, RVC38, RVC39: 49, rcl:R-US_R0603
- added RVC20, RVC21, RVC22, RVC23, RVC24, RVC25, RVC26, RVC27, RVC28, RVC29, RVC30: 100, rcl:R-US_R0603
- added RVC35, RVC37: 1k, rcl:R-US_R0603
- added X4, X5: 5566-12, con-molex:5566-12
- added X6: 5566-16, con-molex:5566-16
- CCB0, CCB1, CCB2, CCB3, CCB4, CCB5, CCB6, CCB7, CCB8, CCB9, CVC0, CVC1, CVC2, CVC3, CVC4, CVC5, CVC6, CVC7, CVC8, CVC9: device rcl:C-EUC0603 -> capacitor-wima:C2.5/2
- RCB0, RCB1, RCB10, RCB2, RCB3, RCB4, RCB5, RCB6, RCB7, RCB8, RCB9: device rcl:R-US_R1210 -> rcl:R-US_R0603
- renumbered CBL to X2, ESDCOML to D1, RBAT to RCB11, RCOML to RVC17, RCOMLN to RVC18, RCOMLP to RVC19, RCOMML to RVC15, RCOMMLN to RVC11, RCOMMLP to RVC12, RNPN to RVC16, TEMPL to X3, TEMPR1 to R8, TEMPR2 to R7, TEMPR3 to R6, TEMPR4 to R5, TEMPR5 to R4, TEMPR6 to R3, TEMPR7 to R2, TEMPR8 to R1, VCL to X1
Connections:
- net CB0 renamed N$25
- net CB1 renamed N$2
- net CB10 renamed N$32
- net CB2 renamed N$4
- net CB3 renamed N$7
- net CB4 renamed N$13
- net CB5 renamed N$16
- net CB6 renamed N$28
- net CB7 renamed N$11
- net CB8 renamed N$19
- net CB9 renamed N$22
- net TEMP1 renamed N$47
- net TEMP2 renamed N$51
- net TEMP3 renamed N$52
- net TEMP4 renamed N$53
- net TEMP5 renamed N$54
- net TEMP6 renamed N$55
- net TEMP7 renamed N$56
- net TEMP8 renamed N$57
- net VC0 renamed N$24
- net VC1 renamed N$1
- net VC10 renamed N$23
- net VC2 renamed N$3
- net VC3 renamed N$9
- net VC4 renamed N$10
- net VC5 renamed N$14
- net VC6 renamed N$26
- net VC7 renamed N$30
- net VC8 renamed N$17
- net VC9 renamed N$20
- removed net CB0-1: CCB0-1.2, IC2.CB0, RCB0-1.2
- removed net CB1-1: CCB0-1.1, CCB1-1.2, IC2.CB1, RCB1-1.2
- removed net CB10-1: CCB9-1.1, IC2.CB10, RCB10-1.2
- removed net CB2-1: CCB1-1.1, CCB2-1.2, IC2.CB2, RCB2-1.2
- removed net CB3-1: CCB2-1.1, CCB3-1.2, IC2.CB3, RCB3-1.2
- removed net CB4-1: CCB3-1.1, CCB4-1.2, IC2.CB4, RCB4-1.2
- removed net CB5-1: CCB4-1.1, CCB5-1.2, IC2.CB5, RCB5-1.2
- removed net CB6-1: CCB5-1.1, CCB6-1.2, IC2.CB6, RCB6-1.2
- removed net CB7-1: CCB6-1.1, CCB7-1.2, IC2.CB7, RCB7-1.2
- removed net CB8-1: CCB7-1.1, CCB8-1.2, IC2.CB8, RCB8-1.2
- removed net CB9-1: CCB8-1.1, CCB9-1.2, IC2.CB9, RCB9-1.2
- removed net COMHN: CCOMHN.1, COMH-2.S
- removed net COMHP: CCOMHP.1, COMH-1.S
- removed net TEMP10: IC2.GPIO2, TEMPH-2.S, TEMPR10.2
- removed net TEMP11: IC2.GPIO3, TEMPH-3.S, TEMPR11.2
- removed net TEMP12: IC2.GPIO4, TEMPH-4.S, TEMPR12.2
- removed net TEMP13: IC2.GPIO5, TEMPH-5.S, TEMPR13.2
- removed net TEMP14: IC2.GPIO6, TEMPH-6.S, TEMPR14.2
- removed net TEMP15: IC2.GPIO7, TEMPH-7.S, TEMPR15.2
- removed net TEMP16: IC2.GPIO8, TEMPH-8.S, TEMPR16.2
- removed net TEMP9: IC2.GPIO1, TEMPH-1.S, TEMPR9.2
- removed net TSREF: CTSREF1.2, IC1.TSREF, R1.1, R2.1, R3.1, R4.1, R5.1, R6.1, R7.1, R8.1
- removed net TSREF-1: CTSREF2.2, IC2.TSREF, TEMPR10.1, TEMPR11.1, TEMPR12.1, TEMPR13.1, TEMPR14.1, TEMPR15.1, TEMPR16.1, TEMPR9.1
- removed net VC0-1: IC2.VC0, RVC0-1.2
- removed net VC1-1: IC2.VC1, RVC1-1.2
- removed net VC10-1: IC2.VC10, RVC10-1.2
- removed net VC2-1: IC2.VC2, RVC2-1.2
- removed net VC3-1: IC2.VC3, RVC3-1.2
- removed net VC4-1: IC2.VC4, RVC4-1.2
- removed net VC5-1: IC2.VC5, RVC5-1.2
- removed net VC6-1: IC2.VC6, RVC6-1.2
- removed net VC7-1: IC2.VC7, RVC7-1.2
- removed net VC8-1: IC2.VC8, RVC8-1.2
- removed net VC9-1: IC2.VC9, RVC9-1.2
- removed net VC_CB_HIGH: CBAT.2, IC1.BAT, IC1.CB11, IC1.CB12, IC1.CB13, IC1.CB14, IC1.CB15, IC1.CB16, IC1.VC11, IC1.VC12, IC1.VC13, IC1.VC14, IC1.VC15, IC1.VC16, RCB11.1
- removed net VC_CB_HIGH-1: CBAT-1.2, IC2.BAT, IC2.CB11, IC2.CB12, IC2.CB13, IC2.CB14, IC2.CB15, IC2.CB16, IC2.VC11, IC2.VC12, IC2.VC13, IC2.VC14, IC2.VC15, IC2.VC16, RBAT-1.1
- new net N$110: CVC17.1, CVC18.2, RVC28.1, X4-10.S
- new net N$115: CCB39.2, IC2.NEG5V
- new net N$116: CCB41.2, IC2.DVDD
- new net N$117: IC2.GPIO1, R16.2, X6-1.S
- new net N$118: IC2.GPIO2, R15.2, X6-2.S
- new net N$119: IC2.GPIO3, R14.2, X6-3.S
- new net N$120: IC2.GPIO4, R13.2, X6-4.S
- new net N$121: IC2.GPIO5, R12.2, X6-5.S
- new net N$122: IC2.GPIO6, R11.2, X6-6.S
- new net N$123: IC2.GPIO7, R10.2, X6-7.S
- new net N$124: IC2.GPIO8, R9.2, X6-8.S
- new net N$127: CCB45.2, IC2.COMHP, RVC32.2, RVC35.1
- new net N$128: CCB42.2, RVC31.1
- new net N$129: CCB43.2, RVC32.1
- new net N$135: CCB50.2, D2.2, RVC39.1
- new net N$136: CCB49.2, D2.1, RVC38.1
- new net N$45: CCB10.2, IC1.BAT, IC1.CB11, IC1.CB12, IC1.CB13, IC1.CB14, IC1.CB15, IC1.CB16, IC1.VC11, IC1.VC12, IC1.VC13, IC1.VC14, IC1.VC15, IC1.VC16, RCB11.1
- new net N$58: C1.2, IC1.TSREF, R1.1, R2.1, R3.1, R4.1, R5.1, R6.1, R7.1, R8.1
- new net N$63: CCB16.1, RVC13.2
- new net N$64: CCB17.1, RVC14.2
- new net N$66: CCB25.1
- new net N$69: CCB24.1
- new net N$70: IC2.VC1, RVC20.2
- new net N$71: CCB26.2, CCB35.1, IC2.CB1, RCB12.2
- new net N$74: RCB13.1, X5-3.S
- new net N$76: CCB27.1, CCB28.2, IC2.CB3, RCB14.2
- new net N$77: RCB14.1, X5-4.S
- new net N$79: IC2.VC4, RVC23.2
- new net N$80: RCB15.1, X5-5.S
- new net N$82: IC2.VC5, RVC24.2
- new net N$83: RCB16.1, X5-6.S
- new net N$85: IC2.VC6, RVC25.2
- new net N$86: RCB17.1, X5-7.S
- new net N$88: IC2.VC7, RVC26.2
- new net N$89: RCB18.1, X5-8.S
- new net N$91: IC2.VC8, RVC27.2
- new net N$92: RCB19.1, X5-9.S
- new net N$94: IC2.VC9, RVC28.2
- new net N$95: RCB20.1, X5-10.S
- new net N$96: CCB33.1, CCB34.2, IC2.CB9, RCB20.2
- new net N$97: IC2.VC10, RVC29.2
- new net N$98: CCB34.1, IC2.CB10, RCB21.2
- net BATC-1: now also RCB21.1, RCB23.2, RVC36.2, X5-11.S; no longer CBH-11.S, RBAT-1.2, RCB10-1.1, RNPN-1.2
- net COMLN: now also CCB49.1; no longer CCOMLN.1
- net COMLP: now also CCB50.1; no longer CCOMLP.1
- net COMMN: now also RVC33.1; no longer CCOMMN.1, RCOMMHN.1
- net COMMP: now also RVC34.1; no longer CCOMMP.1, RCOMMHP.1
- net CVDD: now also CCB14.2; no longer CCVDD.2
- net CVDD-1: now also CCB40.2; no longer CCVDD-1.2
- net GND: now also CCB11.1, CCB12.1, CCB13.1, CCB14.1, CCB15.1, CCB18.2, CCB19.1, CCB21.1, CCB22.1, CCB23.1, IC1.AVSS, IC1.AVSS?, IC1.CVSS, IC1.DVSS, IC1.REFHM; no longer CCOMLNG.1, CCOMLPG.1, CNPN1.1
- net GND-1: now also CCB37.1, CCB38.1, CCB39.1, CCB40.1, CCB41.1, CCB44.2, CCB45.1, CCB47.1, CCB48.1, CCB51.1, D2.3, IC2.AVSS, IC2.AVSS?, IC2.CVSS, IC2.DVSS, IC2.REFHM; no longer CCOMHNG.1, CCOMHPG.1, CNPN1-1.1, ESDCOMH.3
- net GND1: now also C1.1, CCB10.1; no longer CBAT.1, CTSREF1.1
- net GND1-1: now also C2.1, CCB36.1, RCB22.1, X5-1.S, X6-10.S, X6-11.S, X6-12.S, X6-13.S, X6-14.S, X6-15.S, X6-16.S, X6-9.S; no longer CBAT-1.1, CBH-1.S, CTSREF2.1, RCB0-1.1, TEMPH-10.S, TEMPH-11.S, TEMPH-12.S, TEMPH-13.S, TEMPH-14.S, TEMPH-15.S, TEMPH-16.S, TEMPH-9.S
- net GNDN: now also CCB20.1; no longer CAVDD.1, CCOMMLN.2, CCOMMLP.1, CCVDD.1, CDVDD.1, CNEG5V.1, CNPN2.1, CREFHP.1, IC1.AVSS, IC1.AVSS?, IC1.CVSS, IC1.DVSS, IC1.REFHM
- net GNDN-1: now also CCB46.1; no longer CAVDD-1.1, CCOMMHN.1, CCOMMHP.2, CCVDD-1.1, CDVDD-1.1, CNEG5V-1.1, CNPN2-1.1, CREFHP-1.1, IC2.AVSS, IC2.AVSS?, IC2.CVSS, IC2.DVSS, IC2.REFHM
- net LDOIN: now also CCB20.2; no longer CNPN2.2
- net LDOIN-1: now also CCB46.2; no longer CNPN2-1.2
- net N$100: now also CCB35.2, IC2.CB0, RCB22.2; no longer CVC0-1.1, CVC1-1.2, RVC1-1.1, VCH-2.S
- net N$101: now also CVC19.2, RVC30.1, X4-1.S; no longer CVC1-1.1, CVC2-1.2, RVC2-1.1, VCH-3.S
- net N$102: now also CVC10.2, CVC19.1, RVC20.1, X4-2.S; no longer CVC2-1.1, CVC3-1.2, RVC3-1.1, VCH-4.S
- net N$103: now also CVC10.1, CVC11.2, RVC21.1, X4-3.S; no longer CVC3-1.1, CVC4-1.2, RVC4-1.1, VCH-5.S
- net N$104: now also CVC11.1, CVC12.2, RVC22.1, X4-4.S; no longer CVC4-1.1, CVC5-1.2, RVC5-1.1, VCH-6.S
- net N$105: now also CVC12.1, CVC13.2, RVC23.1, X4-5.S; no longer CVC5-1.1, CVC6-1.2, RVC6-1.1, VCH-7.S
- net N$106: now also CVC13.1, CVC14.2, RVC24.1, X4-6.S; no longer CVC6-1.1, CVC7-1.2, RVC7-1.1, VCH-8.S
- net N$107: now also CVC14.1, CVC15.2, RVC25.1, X4-7.S; no longer CVC7-1.1, CVC8-1.2, RVC8-1.1, VCH-9.S
- net N$108: now also CVC15.1, CVC16.2, RVC26.1, X4-8.S; no longer CVC8-1.1, CVC9-1.2, RVC9-1.1, VCH-10.S
- net N$109: now also CVC16.1, CVC17.2, RVC27.1, X4-9.S; no longer CVC9-1.1, RVC10-1.1, VCH-11.S
- net N$111: now also CVC18.1, RVC29.1, X4-11.S; no longer CREFHP-1.2, IC2.REFHP
- net N$112: now also CCB36.2, IC2.BAT, IC2.CB11, IC2.CB12, IC2.CB13, IC2.CB14, IC2.CB15, IC2.CB16, IC2.VC11, IC2.VC12, IC2.VC13, IC2.VC14, IC2.VC15, IC2.VC16, RCB23.1; no longer CAVDD-1.2, IC2.AVDD
- net N$113: now also CCB37.2, IC2.REFHP; no longer CNEG5V-1.2, IC2.NEG5V
- net N$114: now also CCB38.2, IC2.AVDD; no longer CDVDD-1.2, IC2.DVDD
- net N$125: now also C2.2, IC2.TSREF, R10.1, R11.1, R12.1, R13.1, R14.1, R15.1, R16.1, R9.1; no longer CCOMMHN.2, IC2.COMLN, RCOMMH.1, RCOMMHN.2
- net N$126: now also CCB44.1, IC2.COMHN, RVC31.2, RVC35.2; no longer CCOMMHP.1, IC2.COMLP, RCOMMH.2, RCOMMHP.2
- net N$130: now also CCB42.1, RVC33.2; no longer CNPN1-1.2, RNPN-1.1, T2.C
- net N$131: now also CCB43.1, RVC34.2; no longer CCOMHPG.2, IC2.COMHP, RCOMH.2, RCOMHP.2
- net N$132: now also CCB47.2, RVC36.1, T2.C; no longer CCOMHNG.2, IC2.COMHN, RCOMH.1, RCOMHN.2
- net N$133: now also CCB48.2, IC2.COMLN, RVC37.1, RVC38.2; no longer CCOMHP.2, ESDCOMH.1, RCOMHP.1
- net N$134: now also CCB51.2, IC2.COMLP, RVC37.2, RVC39.2; no longer CCOMHN.2, ESDCOMH.2, RCOMHN.1
- net N$29: now also CCB22.2; no longer CCOMLNG.2
- net N$33: now also CCB11.2; no longer CREFHP.2
- net N$46: now also CCB12.2; no longer CAVDD.2
- net N$48: now also CCB13.2; no longer CNEG5V.2
- net N$49: now also CCB23.2; no longer CCOMLPG.2
- net N$50: now also CCB15.2; no longer CDVDD.2
- net N$59: now also CCB18.1; no longer CCOMMLN.1
- net N$60: now also CCB19.2; no longer CCOMMLP.2
- net N$61: now also CCB16.2; no longer CCOMMN.2
- net N$62: now also CCB17.2; no longer CCOMMP.2
- net N$65: now also CCB21.2; no longer CNPN1.2
- net N$67: now also CCB25.2; no longer CCOMLP.2
- net N$68: now also CCB24.2; no longer CCOMLN.2
- net N$72: now also IC2.VC2, RVC21.2; no longer CBH-3.S, RCB2-1.1
- net N$73: now also CCB26.1, CCB27.2, IC2.CB2, RCB13.2; no longer CBH-2.S, RCB1-1.1
- net N$75: now also RCB12.1, X5-2.S; no longer CBH-4.S, RCB3-1.1
- net N$78: now also IC2.VC3, RVC22.2; no longer CBH-5.S, RCB4-1.1
- net N$81: now also CCB28.1, CCB29.2, IC2.CB4, RCB15.2; no longer CBH-6.S, RCB5-1.1
- net N$84: now also CCB29.1, CCB30.2, IC2.CB5, RCB16.2; no longer CBH-7.S, RCB6-1.1
- net N$87: now also CCB30.1, CCB31.2, IC2.CB6, RCB17.2; no longer CBH-8.S, RCB7-1.1
- net N$90: now also CCB31.1, CCB32.2, IC2.CB7, RCB18.2; no longer CBH-9.S, RCB8-1.1
- net N$93: now also CCB32.1, CCB33.2, IC2.CB8, RCB19.2; no longer CBH-10.S, RCB9-1.1
- net N$99: now also IC2.VC0, RVC30.2; no longer CVC0-1.2, RVC0-1.1, VCH-1.S
