File: Hardware/Main Controller/esp_teensy_bridge.brd (EAGLE design)
At the start: 100 x 80 mm, 55 parts, among them IC1 BQ79600PWRQ1, Q1 SI7611DN-T1-GE3, Q2 SI7611DN-T1-GE3, Q3 SI7611DN-T1-GE3

Commit message: layout changes to main
Parts:
- removed R1, R3: 10k ohm, rcl:0204V
- removed R2: 100k ohms, rcl:0204/7
- removed R4: 10km, rcl:0204V
- added R5, R6, R7: 10k, rcl:R0603
- added R8: 100k, rcl:R0603
- moved COML2 101.3 mm to (-66.0, 58.4)
- moved RCOMH 100.8 mm to (-63.5, 33.0)
- moved RCOMHP 100.8 mm to (-73.7, 33.0)
- moved CCOMHN 100.8 mm to (-61.0, 43.2)
- moved CCOMHNG 100.8 mm to (-73.7, 48.3)
- moved CCOMHP 100.8 mm to (-62.2, 38.1)
- moved CCOMHPG 100.8 mm to (-73.7, 43.2)
- moved ESDCOMH 100.8 mm to (-68.6, 27.9)
- moved RCOMHN 100.8 mm to (-73.7, 38.1)
- moved CCOMLNG 81.0 mm to (-27.9, 66.0)
- moved CCB3 79.9 mm to (7.62, 61.0)
- moved CONTACTOR_PRECHARGE 78.2 mm to (92.7, 6.35), turned to 180 degrees
- moved C3 77.5 mm to (33.0, 61.0)
- moved CCB4 73.9 mm to (14.0, 61.0)
- moved COML1 73.8 mm to (-47.0, 58.4)
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Connections:
- net CONTACTORN_CTRL: now also R5.2; no longer R1.2
- net CONTACTORPRECHARGE_CTRL: now also R7.2; no longer R4.2
- net CONTACTORP_CTRL: now also R6.2; no longer R3.2
- net GND: now also R5.1, R6.1, R7.1, R8.2; no longer R1.1, R2.2, R3.1, R4.1
- net N$4: now also R8.1; no longer R2.1

Commit message: fixed some inconsistencies
Parts:
- removed CCB1, CCB22, CCB23, CCB4: 220 pF, capacitor-wima:C2.5-2
- removed CCB2, CCB24, CCB25, CCB3: 2.2nf, capacitor-wima:C2.5-2
- removed COMH, COML: 5566-2, con-molex:5566-2
- removed RVC1, RVC17: 1k, rcl:R0603
- removed RVC18, RVC19, RVC2, RVC3: 49, rcl:R0603
- moved CONTACTOR_P 153.1 mm to (-76.2, 59.7), turned to 0 degrees
- moved Q3 151.6 mm to (-44.5, 85.1), turned to 0 degrees
- moved CONTACTOR_N 147.2 mm to (-57.1, 59.7), turned to 0 degrees
- moved TME1205S 140.5 mm to (-77.5, 40.6), turned to 0 degrees
- moved CONTACTOR_PRECHARGE 140.1 mm to (-36.8, 59.7), turned to 0 degrees
- moved Q1 120.8 mm to (-21.6, 85.1), turned to 0 degrees
- moved Q2 119.8 mm to (-33.0, 85.1), turned to 0 degrees
- moved C3 117.3 mm to (-83.8, 71.1)
- moved CAN 113.3 mm to (-59.7, 41.9), turned to 0 degrees
- moved U$1 109.3 mm to (-31.8, 43.2), turned to 0 degrees
- moved IC1 104.1 mm to (-55.9, 83.8)
- moved ESDCOMH 88.1 mm to (-20.3, 101.6)
- moved PWR_IN 77.5 mm to (-44.5, 73.7)
- moved ESDCOML 69.5 mm to (-35.6, 101.6)
- moved R6 65.6 mm to (-76.2, 96.5)
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Connections:
- removed net N$6: CCB3.2, RVC3.1
- removed net N$66: CCB25.1, COMH.2
- removed net N$67: CCB25.2, RVC19.1
- removed net N$68: CCB24.2, RVC18.1
- removed net N$69: CCB24.1, COMH.1
- removed net N$7: CCB2.2, RVC2.1
- removed net N$8: CCB2.1, COML.1
- removed net N$9: CCB3.1, COML.2
- net COMHN: no longer CCB22.2, RVC17.1, RVC18.2
- net COMHP: no longer CCB23.2, RVC17.2, RVC19.2
- net COMLN: no longer CCB4.2, RVC1.2, RVC3.2
- net COMLP: no longer CCB1.2, RVC1.1, RVC2.2
- net GND: no longer CCB1.1, CCB22.1, CCB23.1, CCB4.1
- net VCC: now also CONTACTOR_N.1, CONTACTOR_P.1, CONTACTOR_PRECHARGE.1
Other:
- board size 100 x 80 mm -> 160 x 100 mm

Commit message: recreated pcb
Parts:
- moved U$2 96.4 mm to (57.1, 48.3), turned to 180 degrees
- moved U$1 51.4 mm to (19.1, 50.8)
Changed lines of the file:
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@@
 <attribute name="VALUE" x="-74.422" y="35.56" size="1.27" layer="27" ratio="10" rot="R90"/>
 </element>
-<element name="U$1" library="teensy" package="TEENSY40" value="TEENSY40" x="-31.75" y="43.18" smashed="yes"/>
-<element name="U$2" library="ESP32-DEVKITV1" package="ESP32-DEVKITV1" value="ESP32DEVKITV1" x="-34.29" y="17.78" smashed="yes">
-<attribute name="NAME" x="-58.42" y="31.75" size="1.27" layer="21"/>
+<element name="U$1" library="teensy" package="TEENSY40" value="TEENSY40" x="19.05" y="50.8" smashed="yes"/>
+<element name="U$2" library="ESP32-DEVKITV1" package="ESP32-DEVKITV1" value="ESP32DEVKITV1" x="57.15" y="48.26" smashed="yes" rot="R180">
+<attribute name="NAME" x="81.28" y="34.29" size="1.27" layer="21" rot="R180"/>
 </element>
 </elements>
@@
 <wire x1="-77.05" y1="96.52" x2="-71.97" y2="96.52" width="0" layer="19" extent="1-1"/>
 <wire x1="-82.13" y1="96.52" x2="-77.05" y2="96.52" width="0" layer="19" extent="1-1"/>
-<wire x1="-45.72" y1="50.8" x2="-54.61" y2="71.12" width="0" layer="19" extent="1-1"/>
-<wire x1="-57.59" y1="44.66" x2="-45.72" y2="50.8" width="0" layer="19" extent="1-1"/>
-<wire x1="-48.26" y1="35.56" x2="-57.59" y2="44.66" width="0" layer="19" extent="1-1"/>
+<wire x1="5.08" y1="58.42" x2="-54.61" y2="71.12" width="0" layer="19" extent="1-1"/>
+<wire x1="-57.59" y1="44.66" x2="5.08" y2="58.42" width="0" layer="19" extent="1-1"/>
+<wire x1="2.54" y1="43.18" x2="-57.59" y2="44.66" width="0" layer="19" extent="1-1"/>
 <wire x1="-77.47" y1="44.45" x2="-57.59" y2="44.66" width="0" layer="19" extent="1-1"/>
 <wire x1="-77.47" y1="39.37" x2="-77.47" y2="44.45" width="0" layer="19" extent="1-1"/>
-<wire x1="-15.24" y1="43.18" x2="-45.72" y2="50.8" width="0" layer="19" extent="1-1"/>
-<wire x1="-54.62" y1="4.24" x2="-48.26" y2="35.56" width="0" layer="19" extent="1-1"/>
+<wire x1="35.56" y1="50.8" x2="5.08" y2="58.42" width="0" layer="19" extent="1-1"/>
+<wire x1="77.48" y1="61.8" x2="2.54" y2="43.18" width="0" layer="19" extent="1-1"/>
 </signal>
 <signal name="NCS/CS">
@@
 <contactref element="U$1" pad="0-RX1"/>
 <contactref element="U$2" pad="13"/>
-<wire x1="-45.72" y1="35.56" x2="-26.68" y2="4.24" width="0" layer="19" extent="1-1"/>
+<wire x1="5.08" y1="43.18" x2="49.54" y2="61.8" width="0" layer="19" extent="1-1"/>
 </signal>
 <signal name="RX_ESP">
 <contactref element="U$1" pad="1-TX1"/>
 <contactref element="U$2" pad="12"/>
-<wire x1="-43.18" y1="35.56" x2="-29.22" y2="4.24" width="0" layer="19" extent="1-1"/>
+<wire x1="7.62" y1="43.18" x2="52.08" y2="61.8" width="0" layer="19" extent="1-1"/>
 </signal>
 <signal name="TX_BRIDGE">
 <contactref element="U$1" pad="28-RX7"/>
 <contactref element="IC1" pad="5"/>
-<wire x1="-58.818" y1="83.495" x2="-19.05" y2="43.18" width="0" layer="19" extent="1-1"/>
+<wire x1="-58.818" y1="83.495" x2="31.75" y2="50.8" width="0" layer="19" extent="1-1"/>
 </signal>
 <signal name="RX_BRIDGE">
 <contactref element="U$1" pad="29-TX7"/>
 <contactref element="IC1" pad="4"/>
-<wire x1="-23.495" y1="43.18" x2="-58.818" y2="84.145" width="0" layer="19" extent="1-1"/>
+<wire x1="27.305" y1="50.8" x2="-58.818" y2="84.145" width="0" layer="19" extent="1-1"/>
 </signal>
 <signal name="5V">
@@
 <contactref element="TME1205S" pad="4"/>
 <contactref element="C5" pad="1"/>
-<wire x1="-57.16" y1="29.01" x2="-77.47" y2="36.83" width="0" layer="19" extent="1-1"/>
-<wire x1="-48.26" y1="50.8" x2="-57.16" y2="29.01" width="0" layer="19" extent="1-1"/>
-<wire x1="-64.77" y1="71.12" x2="-48.26" y2="50.8" width="0" layer="19" extent="1-1"/>
+<wire x1="80.02" y1="37.03" x2="-77.47" y2="36.83" width="0" layer="19" extent="1-1"/>
+<wire x1="2.54" y1="58.42" x2="80.02" y2="37.03" width="0" layer="19" extent="1-1"/>
+<wire x1="-64.77" y1="71.12" x2="2.54" y2="58.42" width="0" layer="19" extent="1-1"/>
 </signal>
 <signal name="VCC">
@@
 <contactref element="U$1" pad="30-CRX3"/>
 <contactref element="CAN" pad="1"/>
-<wire x1="-57.59" y1="39.16" x2="-19.05" y2="40.64" width="0" layer="19" extent="1-1"/>
+<wire x1="-57.59" y1="39.16" x2="31.75" y2="48.26" width="0" layer="19" extent="1-1"/>
 </signal>
 <signal name="CTX">
 <contactref element="U$1" pad="31-CTX3"/>
 <contactref element="CAN" pad="2"/>
-<wire x1="-23.495" y1="40.64" x2="-61.79" y2="39.16" width="0" layer="19" extent="1-1"/>
+<wire x1="27.305" y1="48.26" x2="-61.79" y2="39.16" width="0" layer="19" extent="1-1"/>
 </signal>
 <signal name="CONTACTORN_CTRL">
@@
 <contactref element="R5" pad="2"/>
 <contactref element="U$1" pad="32-OUTB1"/>
-<wire x1="-19.05" y1="38.1" x2="-23.025" y2="84.1" width="0" layer="19" extent="1-1"/>
+<wire x1="31.75" y1="45.72" x2="-23.025" y2="84.1" width="0" layer="19" extent="1-1"/>
 <wire x1="-70.27" y1="96.52" x2="-23.025" y2="84.1" width="0" layer="19" extent="1-1"/>
 </signal>
@@
 <contactref element="U$1" pad="9-OUT1C"/>
 <wire x1="-75.35" y1="96.52" x2="-34.455" y2="84.1" width="0" layer="19" extent="1-1"/>
-<wire x1="-22.86" y1="35.56" x2="-34.455" y2="84.1" width="0" layer="19" extent="1-1"/>
+<wire x1="27.94" y1="43.18" x2="-34.455" y2="84.1" width="0" layer="19" extent="1-1"/>
 </signal>
 <signal name="CONTACTORPRECHARGE_CTRL">
@@
 <contactref element="U$1" pad="6-OUT1D"/>
 <wire x1="-80.43" y1="96.52" x2="-45.885" y2="84.1" width="0" layer="19" extent="1-1"/>
-<wire x1="-30.48" y1="35.56" x2="-45.885" y2="84.1" width="0" layer="19" extent="1-1"/>
+<wire x1="20.32" y1="43.18" x2="-45.885" y2="84.1" width="0" layer="19" extent="1-1"/>
 </signal>
 <signal name="N$12">

Commit message: 12/1/2021
Parts:
- added COOLANT-1: 5566-2, con-molex:5566-2
- added Q4: SI7611DN-T1-GE3, SI7611DN-T1-GE3:VISHAY_SIS468DN-T1-GE3
- added R1: 10k, rcl:R0603
Connections:
- new net COOLANT_CTRL: Q4.4, R1.2
- new net N$6: COOLANT-1.2, Q4.1, Q4.2, Q4.3
- net GND: now also Q4.5, Q4.6, Q4.7, Q4.8, Q4.9, R1.1
- net VCC: now also COOLANT-1.1
Changed lines of the file:
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@@
 <attribute name="NAME" x="81.28" y="34.29" size="1.27" layer="21" rot="R180"/>
+</element>
+<element name="COOLANT-1" library="con-molex" library_urn="urn:adsk.eagle:library:165" package="5566-2" package3d_urn="urn:adsk.eagle:package:8078583/1" value="5566-2" x="-80.01" y="-7.62" smashed="yes">
+<attribute name="MF" value="MOLEX" x="-93.98" y="7.62" size="1.778" layer="27" display="off"/>
+<attribute name="MPN" value="" x="-93.98" y="7.62" size="1.778" layer="27" display="off"/>
+<attribute name="NAME" x="-81.28" y="-2.54" size="1.27" layer="25"/>
+<attribute name="OC_FARNELL" value="1822072" x="-93.98" y="7.62" size="1.778" layer="27" display="off"/>
+<attribute name="OC_NEWARK" value="unknown" x="-93.98" y="7.62" size="1.778" layer="27" display="off"/>
+<attribute name="POPULARITY" value="0" x="-93.98" y="7.62" size="1.778" layer="27" display="off"/>
+<attribute name="VALUE" x="-82.55" y="-13.97" size="1.27" layer="27"/>
+</element>
+<element name="Q4" library="SI7611DN-T1-GE3" package="VISHAY_SIS468DN-T1-GE3" value="SI7611DN-T1-GE3" x="-83.82" y="-17.78" smashed="yes">
+<attribute name="AVAILABILITY" value="In Stock" x="-102.87" y="3.81" size="1.778" layer="27" display="off"/>
+<attribute name="DESCRIPTION" value=" P-Channel 40 V 18A (Tc) 3.7W (Ta), 39W (Tc) Surface Mount PowerPAK® 1212-8 " x="-102.87" y="3.81" size="1.778" layer="27" display="off"/>
+<attribute name="MF" value="Vishay Siliconix" x="-102.87" y="3.81" size="1.778" layer="27" display="off"/>
+<attribute name="MP" value="SI7611DN-T1-GE3" x="-102.87" y="3.81" size="1.778" layer="27" display="off"/>
+<attribute name="NAME" x="-86.074459375" y="-15.77603125" size="0.81343125" layer="25"/>
+<attribute name="PACKAGE" value="PowerPAK®-1212 Vishay" x="-102.87" y="3.81" size="1.778" layer="27" display="off"/>
+<attribute name="PRICE" value="None" x="-102.87" y="3.81" size="1.778" layer="27" display="off"/>
+<attribute name="PURCHASE-URL" value="https://pricing.snapeda.com/search/part/SI7611DN-T1-GE3/?ref=eda" x="-102.87" y="3.81" size="1.778" layer="27" display="off"/>
+<attribute name="VALUE" x="-86.07581875" y="-20.738340625" size="0.812984375" layer="27"/>
+</element>
+<element name="R1" library="rcl" library_urn="urn:adsk.eagle:library:334" package="R0603" package3d_urn="urn:adsk.eagle:package:23555/3" value="10k" x="-73.66" y="-17.78" smashed="yes">
+<attribute name="NAME" x="-74.295" y="-17.145" size="1.27" layer="25"/>
+<attribute name="POPULARITY" value="77" x="-102.87" y="-2.54" size="1.778" layer="27" display="off"/>
+<attribute name="SPICEPREFIX" value="R" x="-102.87" y="-2.54" size="1.778" layer="27" display="off"/>
+<attribute name="VALUE" x="-74.295" y="-19.685" size="1.27" layer="27"/>
 </element>
 </elements>
@@
 <contactref element="ESDCOML" pad="3"/>
 <contactref element="ESDCOMH" pad="3"/>
-<wire x1="-34.41" y1="101.6" x2="-19.17" y2="101.6" width="0" layer="19" extent="1-1"/>
-<wire x1="-20.04" y1="86.08" x2="-19.17" y2="101.6" width="0" layer="19" extent="1-1"/>
-<wire x1="-20.04" y1="85.42" x2="-20.04" y2="86.08" width="0" layer="19" extent="1-1"/>
-<wire x1="-20.04" y1="84.76" x2="-20.04" y2="85.42" width="0" layer="19" extent="1-1"/>
-<wire x1="-20.04" y1="84.1" x2="-20.04" y2="84.76" width="0" layer="19" extent="1-1"/>
-<wire x1="-21.0325" y1="85.09" x2="-20.04" y2="85.42" width="0" layer="19" extent="1-1"/>
+<contactref element="Q4" pad="9"/>
+<contactref element="Q4" pad="7"/>
+<contactref element="Q4" pad="6"/>
+<contactref element="Q4" pad="5"/>
+<contactref element="Q4" pad="8"/>
+<contactref element="R1" pad="1"/>
+<wire x1="35.56" y1="50.8" x2="77.48" y2="61.8" width="0" layer="19" extent="1-1"/>
+<wire x1="5.08" y1="58.42" x2="35.56" y2="50.8" width="0" layer="19" extent="1-1"/>
+<wire x1="2.54" y1="43.18" x2="5.08" y2="58.42" width="0" layer="19" extent="1-1"/>
+<wire x1="-20.04" y1="84.1" x2="5.08" y2="58.42" width="0" layer="19" extent="1-1"/>
+<wire x1="-20.04" y1="84.76" x2="-20.04" y2="84.1" width="0" layer="19" extent="1-1"/>
+<wire x1="-20.04" y1="85.42" x2="-20.04" y2="84.76" width="0" layer="19" extent="1-1"/>
+<wire x1="-20.04" y1="86.08" x2="-20.04" y2="85.42" width="0" layer="19" extent="1-1"/>
+<wire x1="-21.0325" y1="85.09" x2="-20.04" y2="84.76" width="0" layer="19" extent="1-1"/>
 <wire x1="-31.47" y1="84.76" x2="-21.0325" y2="85.09" width="0" layer="19" extent="1-1"/>
 <wire x1="-31.47" y1="84.1" x2="-31.47" y2="84.76" width="0" layer="19" extent="1-1"/>
@@
 <wire x1="-77.05" y1="96.52" x2="-71.97" y2="96.52" width="0" layer="19" extent="1-1"/>
 <wire x1="-82.13" y1="96.52" x2="-77.05" y2="96.52" width="0" layer="19" extent="1-1"/>
-<wire x1="5.08" y1="58.42" x2="-54.61" y2="71.12" width="0" layer="19" extent="1-1"/>
-<wire x1="-57.59" y1="44.66" x2="5.08" y2="58.42" width="0" layer="19" extent="1-1"/>
-<wire x1="2.54" y1="43.18" x2="-57.59" y2="44.66" width="0" layer="19" extent="1-1"/>
+<wire x1="-19.17" y1="101.6" x2="-20.04" y2="86.08" width="0" layer="19" extent="1-1"/>
+<wire x1="-34.41" y1="101.6" x2="-19.17" y2="101.6" width="0" layer="19" extent="1-1"/>
+<wire x1="-57.59" y1="44.66" x2="-54.61" y2="71.12" width="0" layer="19" extent="1-1"/>
 <wire x1="-77.47" y1="44.45" x2="-57.59" y2="44.66" width="0" layer="19" extent="1-1"/>
 <wire x1="-77.47" y1="39.37" x2="-77.47" y2="44.45" width="0" layer="19" extent="1-1"/>
-<wire x1="35.56" y1="50.8" x2="5.08" y2="58.42" width="0" layer="19" extent="1-1"/>
-<wire x1="77.48" y1="61.8" x2="2.54" y2="43.18" width="0" layer="19" extent="1-1"/>
+<wire x1="-82.27" y1="-16.79" x2="-77.47" y2="39.37" width="0" layer="19" extent="1-1"/>
+<wire x1="-82.27" y1="-17.45" x2="-82.27" y2="-16.79" width="0" layer="19" extent="1-1"/>
+<wire x1="-82.27" y1="-18.11" x2="-82.27" y2="-17.45" width="0" layer="19" extent="1-1"/>
+<wire x1="-82.27" y1="-18.77" x2="-82.27" y2="-18.11" width="0" layer="19" extent="1-1"/>
+<wire x1="-83.2625" y1="-17.78" x2="-82.27" y2="-17.45" width="0" layer="19" extent="1-1"/>
+<wire x1="-74.51" y1="-17.78" x2="-82.27" y2="-17.45" width="0" layer="19" extent="1-1"/>
 </signal>
 <signal name="NCS/CS">
@@
 <contactref element="CONTACTOR_P" pad="1"/>
 <contactref element="CONTACTOR_PRECHARGE" pad="1"/>
+<contactref element="COOLANT-1" pad="1"/>
+<wire x1="-77.47" y1="41.91" x2="-80.01" y2="-10.37" width="0" layer="19" extent="1-1"/>
 <wire x1="-76.2" y1="56.94" x2="-77.47" y2="41.91" width="0" layer="19" extent="1-1"/>
 <wire x1="-77.47" y1="71.12" x2="-76.2" y2="56.94" width="0" layer="19" extent="1-1"/>
@@
 <contactref element="R7" pad="2"/>
 <contactref element="U$1" pad="6-OUT1D"/>
+<wire x1="-45.885" y1="84.1" x2="20.32" y2="43.18" width="0" layer="19" extent="1-1"/>
 <wire x1="-80.43" y1="96.52" x2="-45.885" y2="84.1" width="0" layer="19" extent="1-1"/>
-<wire x1="20.32" y1="43.18" x2="-45.885" y2="84.1" width="0" layer="19" extent="1-1"/>
 </signal>
 <signal name="N$12">
@@
 <wire x1="-66.89" y1="96.52" x2="-52.942" y2="86.095" width="0" layer="19" extent="1-1"/>
 </signal>
+<signal name="N$6">
+<contactref element="Q4" pad="1"/>
+<contactref element="Q4" pad="2"/>
+<contactref element="Q4" pad="3"/>
+<contactref element="COOLANT-1" pad="2"/>
+<wire x1="-85.255" y1="-17.45" x2="-85.255" y2="-18.11" width="0" layer="19" extent="1-1"/>
+<wire x1="-85.255" y1="-16.79" x2="-85.255" y2="-17.45" width="0" layer="19" extent="1-1"/>
+<wire x1="-80.01" y1="-4.87" x2="-85.255" y2="-16.79" width="0" layer="19" extent="1-1"/>
+</signal>
+<signal name="COOLANT_CTRL">
+<contactref element="Q4" pad="4"/>
+<contactref element="R1" pad="2"/>
+<wire x1="-72.81" y1="-17.78" x2="-85.255" y2="-18.77" width="0" layer="19" extent="1-1"/>
+</signal>
 </signals>

Commit message: have fun with eagle
Parts:
- C1, C2, C4, C5: device capacitor-wima:C2.5-3 -> rcl:C0603
- C3: device capacitor-wima:C2.5-2 -> rcl:C0603
- moved CAN 115.1 mm to (49.5, 78.1)
- moved CONTACTOR_N 94.0 mm to (34.9, 78.7)
- moved COOLANT-1 67.1 mm to (-39.4, 45.7)
- moved Q4 67.1 mm to (-43.2, 35.6)
- moved R1 67.1 mm to (-33.0, 35.6)
- moved CONTACTOR_P 64.3 mm to (-15.2, 80.0)
- moved Q1 57.8 mm to (34.3, 70.5)
- moved Q2 55.9 mm to (21.0, 70.5)
- moved Q3 54.7 mm to (8.26, 70.5)
- moved PWR_IN 41.3 mm to (-8.89, 94.6), turned to 180 degrees
- moved RCOMHP 37.0 mm to (-54.0, 61.0)
- moved CCOMHPG 35.6 mm to (-62.2, 56.5)
- moved IC1 30.1 mm to (-69.8, 57.1)
- moved COML2 27.6 mm to (-18.4, 49.5)
- moved CCOMHNG 26.7 mm to (-62.2, 59.7)
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Other:
- board size 160 x 100 mm -> 100.3 x 100.6 mm

Commit message: placed some wires
Parts:
- removed CAN: 5566-4, con-molex:5566-4
- removed COML1, COML2: 5566-2, con-molex:5566-2
- removed U$1: TEENSY40, teensy:TEENSY40
- added CAN1: 5566-4, con-molex:5566-4
- added COMH, COML: 5566-2, con-molex:5566-2
- added U$3: TEENSY41, teensy:TEENSY41
- moved C5 221.6 mm to (154.3, 50.2)
- moved C4 204.5 mm to (132.1, 58.4)
- moved C1 204.5 mm to (142.9, 60.3)
- moved CCOMHNG 204.5 mm to (142.2, 55.2)
- moved CCOMHPG 204.5 mm to (142.2, 52.1)
- moved RCOMHP 204.5 mm to (150.5, 56.5)
- moved C3 204.5 mm to (137.8, 58.4)
- moved CCOMHN 193.7 mm to (149.2, 91.4)
- moved CCOMHP 193.7 mm to (128.9, 91.4)
- moved CCOMLP 193.7 mm to (161.9, 96.5)
- moved RCOMH 193.7 mm to (142.9, 96.5)
- moved RCOMHN 193.7 mm to (139.1, 91.4)
- moved RCOML 193.7 mm to (134.0, 96.5)
- moved CCOMLPG 193.7 mm to (159.4, 91.4)
- moved RCOMLP 193.7 mm to (151.8, 96.5)
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Connections:
- removed net CRX: CAN.1, U$1.30-CRX3
- removed net CTX: CAN.2, U$1.31-CTX3
- new net N$7: CAN1.1, U$3.30-CRX3
- new net N$8: CAN1.2, U$3.31-CTX3
- net 5V: now also U$3.VIN; no longer U$1.VIN
- net COMHN_ISO: now also COMH.1; no longer COML2.1
- net COMHP_ISO: now also COMH.2; no longer COML2.2
- net COMLN_ISO: now also COML.1; no longer COML1.1
- net COMLP_ISO: now also COML.2; no longer COML1.2
- net CONTACTORN_CTRL: now also U$3.23-A9/CRX1/MCLK1; no longer U$1.32-OUTB1
- net CONTACTORPRECHARGE_CTRL: now also U$3.21-A7/RX5/BCLK1; no longer U$1.6-OUT1D
- net CONTACTORP_CTRL: now also U$3.22-A8/CTX1; no longer U$1.9-OUT1C
- net COOLANT_CTRL: now also U$3.20-A6/TX5/LRCLK1
- net GND: now also CAN1.3, U$3.GND1, U$3.GND2, U$3.GND3; no longer CAN.3, U$1.GND1, U$1.GND2, U$1.GND3
- net NCS/CS: now also U$3.10-CS\MQSR; no longer U$1.10-CS/MQSR
- net RX_BRIDGE: now also U$3.29-TX7; no longer U$1.29-TX7
- net RX_ESP: now also U$3.1-TX1/MISO1/CTX2; no longer U$1.1-TX1
- net TX_BRIDGE: now also U$3.28-RX7; no longer U$1.28-RX7
- net TX_ESP: now also U$3.0-RX1/CS1/CRX2; no longer U$1.0-RX1
- net VCC: now also PWR_IN.1
Routing:
- net VCC: track 0.00 -> 76.1 mm
- net N$6: track 0.00 -> 6.43 mm
- net N$2: track 0.00 -> 6.43 mm
- net N$5: track 0.00 -> 6.43 mm
- net N$12: track 0.00 -> 6.43 mm
- net COOLANT_CTRL: track 0.00 -> 3.70 mm
- net CONTACTORP_CTRL: track 0.00 -> 3.70 mm
- net CONTACTORN_CTRL: track 0.00 -> 3.70 mm
- net CONTACTORPRECHARGE_CTRL: track 0.00 -> 3.70 mm

Commit message: 1/8/2022
Parts:
- moved CCOMLN 145.6 mm to (60.3, 84.5)
- moved CAN1 133.3 mm to (64.8, 52.1), turned to 180 degrees
- moved C5 99.4 mm to (59.7, 19.7)
- moved CCOMLP 98.3 mm to (64.8, 81.3)
- moved ESDCOML 92.3 mm to (67.9, 63.5)
- moved RCOMLP 92.0 mm to (81.3, 37.5)
- moved RCOMHP 91.6 mm to (64.8, 24.1)
- moved COMH 91.2 mm to (94.0, 43.8)
- moved CCOMLPG 90.4 mm to (91.4, 31.8), turned to 180 degrees
- moved CCOMLNG 88.9 mm to (84.5, 58.4)
- moved C1 88.0 mm to (64.8, 19.7), turned to 180 degrees
- moved RCOMH 87.9 mm to (86.4, 29.2)
- moved RCOMHN 86.3 mm to (81.3, 27.3)
- moved CCOMHN 84.9 mm to (87.0, 33.7)
- moved R8 84.9 mm to (63.5, 41.9)
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Routing:
- net 5V: track 0.00 -> 102.3 mm, vias 0 -> 1
- net GND: track 0.00 -> 96.8 mm, vias 0 -> 4
- net COOLANT_CTRL: track 3.70 -> 29.6 mm
- net CONTACTORPRECHARGE_CTRL: track 3.70 -> 19.4 mm
- net TX_ESP: track 0.00 -> 12.5 mm
- net RX_ESP: track 0.00 -> 12.5 mm
- net CONTACTORN_CTRL: track 3.70 -> 13.5 mm
- net VCC: track 76.1 -> 84.1 mm
- net CONTACTORP_CTRL: track 3.70 -> 11.3 mm
Other:
- board size 100.3 x 100.6 mm -> 102.8 x 87.9 mm
