File: Hardware/Main controller 79656/esp_teensy_bridge.brd (EAGLE design)
At the start: 99.8 x 88.1 mm, 105 parts, among them IC2 PBQ79656PAPTQ1, Q5 VISHAY_SIS862DN-T1-GE3VISHAY_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, Q6 VISHAY_SIS862DN-T1-GE3VISHAY_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, Q7 VISHAY_SIS862DN-T1-GE3VISHAY_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, Q8 VISHAY_SIS862DN-T1-GE3VISHAY_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, T2 PBHV8115X, 115, U1 MCP2562-E/SN, U2 ESP32-DEVKITC-32D, X1 5566-12

Commit message: level shiffft
Parts:
- added U$1: TXB0108PWSMD, TB0108:TSSOP20
Connections:
- new net RX_SHFT: U$1.18, U$3.34-RX8
- new net TX_SHFT: U$1.20, U$3.35-TX8
- new net VCCB: U$1.19
- net 3V3: now also U$1.2
- net GND: now also U$1.11
- net RX_BQ: now also U$1.3; no longer U$3.35-TX8
- net TX_BQ: now also U$1.1; no longer U$3.34-RX8
Changed lines of the file:
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@@
 <attribute name="VALUE" x="-21.717" y="-145.288" size="1.27" layer="27"/>
+</element>
+<element name="U$1" library="TB0108" package="TSSOP20" value="TXB0108PWSMD" x="34.798" y="-23.114" smashed="yes" rot="R270">
+<attribute name="NAME" x="32.7152" y="-19.5684" size="1.016" layer="25" ratio="10"/>
+<attribute name="VALUE" x="32.7152" y="-27.6502" size="1.016" layer="27" ratio="10"/>
 </element>
 </elements>
@@
 <contactref element="RCB0-1" pad="1"/>
 <contactref element="R2" pad="1"/>
+<contactref element="U$1" pad="11"/>
+<wire x1="-22.032" y1="-129.794" x2="37.7158" y2="-26.039" width="0" layer="19" extent="1-1"/>
 <wire x1="-0.628" y1="-91.948" x2="-22.032" y2="-129.794" width="0" layer="19" extent="1-1"/>
 <wire x1="0.674" y1="-67.31" x2="-0.628" y2="-91.948" width="0" layer="19" extent="1-1"/>
@@
 <wire x1="45.72" y1="40.64" x2="46.43" y2="40.64" width="0.3048" layer="16"/>
 <wire x1="46.43" y1="40.64" x2="48.97" y2="38.1" width="0.3048" layer="16"/>
+<contactref element="U$1" pad="2"/>
+<wire x1="58.205" y1="21.805" x2="31.8802" y2="-20.839" width="0" layer="19" extent="1-1"/>
 </signal>
 <signal name="CRX">
@@
 </signal>
 <signal name="TX_BQ">
-<contactref element="U$3" pad="34-RX8"/>
 <contactref element="IC2" pad="53"/>
-<wire x1="13.434" y1="-29.314" x2="57.785" y2="62.5475" width="0" layer="19" extent="1-1"/>
+<contactref element="U$1" pad="1"/>
+<wire x1="13.434" y1="-29.314" x2="31.8802" y2="-20.189" width="0" layer="19" extent="1-1"/>
 </signal>
 <signal name="RX_BQ">
-<contactref element="U$3" pad="35-TX8"/>
 <contactref element="IC2" pad="52"/>
-<wire x1="13.934" y1="-29.314" x2="55.245" y2="62.5475" width="0" layer="19" extent="1-1"/>
+<contactref element="U$1" pad="3"/>
+<wire x1="13.934" y1="-29.314" x2="31.8802" y2="-21.489" width="0" layer="19" extent="1-1"/>
 </signal>
 <signal name="VC1-1">
@@
 <wire x1="-3.048" y1="-98.088" x2="0.674" y2="-115.316" width="0" layer="19" extent="1-1"/>
 </signal>
+<signal name="RX_SHFT">
+<contactref element="U$3" pad="34-RX8"/>
+<contactref element="U$1" pad="18"/>
+<wire x1="57.785" y1="62.5475" x2="37.7158" y2="-21.489" width="0" layer="19" extent="1-1"/>
+</signal>
+<signal name="TX_SHFT">
+<contactref element="U$3" pad="35-TX8"/>
+<contactref element="U$1" pad="20"/>
+<wire x1="55.245" y1="62.5475" x2="37.7158" y2="-20.189" width="0" layer="19" extent="1-1"/>
+</signal>
+<signal name="VCCB">
+<contactref element="U$1" pad="19"/>
+</signal>
 </signals>

Commit message: Late night mainboard layout
Parts:
- removed CCB0-1, CCB1-1, CCB2-1, CCB3-1: 0.47uf, rcl:C0603
- removed GNDH: (no value), wirepad:SMD2,54-5,08
- removed RCB0-1, RCB1-1, RCB2-1, RCB3-1, RCB4-1: 10, rcl:R1210
- moved R9 183.9 mm to (58.4, 23.1), turned to 90 degrees
- moved R4 176.2 mm to (58.4, 18.8), turned to 90 degrees
- moved R3 168.5 mm to (58.4, 14.5), turned to 90 degrees
- moved TEMPR9 157.9 mm to (85.3, 55.1)
- moved R2 156.7 mm to (52.3, 8.64), turned to 90 degrees
- moved RCOMLP 149.1 mm to (71.1, 6.10)
- moved RCOML 146.5 mm to (73.9, 6.86), turned to 90 degrees
- moved ESDCOML 146.3 mm to (69.1, 3.30), turned to 180 degrees
- moved RCOMLN 142.3 mm to (72.9, 1.78)
- moved CCOMLPG 142.0 mm to (70.6, 8.13)
- moved CCOMLP 136.2 mm to (65.3, 5.08)
- moved RVC4-1 131.8 mm to (62.0, 24.1)
- moved TEMPR15 130.4 mm to (85.1, 29.2)
- moved CCOMLN 128.0 mm to (65.3, 1.52)
- moved ESDCOMH 126.8 mm to (80.8, 4.32)
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Connections:
- removed net BATC-1: RNPN-1.2
- removed net CB0-1: CCB0-1.2, IC2.34, RCB0-1.2
- removed net CB1-1: CCB0-1.1, CCB1-1.2, IC2.32, RCB1-1.2
- removed net CB2-1: CCB1-1.1, CCB2-1.2, IC2.30, RCB2-1.2
- removed net CB3-1: CCB2-1.1, CCB3-1.2, IC2.28, RCB3-1.2
- removed net CB4-1: CCB10-1.1, CCB3-1.1, IC2.26, RCB4-1.2
- removed net N$125: IC2.41
- removed net N$126: IC2.40
- removed net VCCB: U$1.19
- net 3V3: now also U$1.10
- net 5V: now also U$1.19
- net GND: no longer GNDH.1, RCB0-1.1
- net N$10: now also IC2.41
- net N$49: now also IC2.40
- net N$72: no longer RCB2-1.1
- net N$73: no longer RCB1-1.1
- net N$75: no longer RCB3-1.1
- net RX_BQ: now also U$1.18; no longer U$1.3
- net RX_SHFT: now also U$1.1; no longer U$1.18
- net TX_BQ: now also U$1.20; no longer U$1.1
- net TX_SHFT: now also U$1.3; no longer U$1.20
- net VC0-1: now also IC2.34
- net VC1-1: now also IC2.32
- net VC2-1: now also IC2.30
- net VC3-1: now also IC2.28
- net VC4-1: now also CCB10-1.1, IC2.26
- net VCC: now also RNPN-1.2; no longer RCB4-1.1
Routing:
- net SPI_RDY: track 81.2 -> 0.00 mm
- net SCK: track 74.6 -> 0.00 mm, vias 4 -> 0
- net CS0: track 64.5 -> 0.00 mm, vias 2 -> 0
- net NFAULT: track 62.8 -> 0.00 mm, vias 1 -> 0
- net MOSI: track 62.5 -> 0.00 mm, vias 2 -> 0
- net MISO: track 60.2 -> 0.00 mm, vias 2 -> 0
- net TEMP9: track 0.00 -> 46.9 mm
- net TEMP10: track 0.00 -> 44.3 mm, vias 0 -> 2
- net TX_SHFT: track 0.00 -> 43.3 mm
- net TSREF-1: track 0.00 -> 42.3 mm, vias 0 -> 2
- net RX_SHFT: track 0.00 -> 42.1 mm
- net TEMP11: track 0.00 -> 34.9 mm, vias 0 -> 2
- net TEMP12: track 0.00 -> 31.4 mm, vias 0 -> 2
- net TEMP13: track 0.00 -> 28.7 mm, vias 0 -> 2
- net GND: track 49.9 -> 74.8 mm, vias 4 -> 7
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- removed copper zone on layer 16, net 5V

Commit message: dc dc buck converter replace
Parts:
- added C1: 2.2μF, rcl:C0603
- added C2: 10μF, rcl:C0603
- added L1: 5.6 uH, inductor-neosid:SD8
- added PWR_IN1: 5566-2, con-molex:5566-2
- added R-78-1.0: (no value), v-reg:78XXS
Connections:
- new net N$16: C1.1, L1.2, R-78-1.0.IN
- new net N$36: C2.1, L1.1, PWR_IN1.1
- net 5V: now also R-78-1.0.OUT
- net GND: now also C1.2, C2.2, PWR_IN1.2, R-78-1.0.GND

Commit message: buck converter layout
Parts:
- removed C4: 0.1μF, rcl:C0603
- removed C5: 0.22μF, rcl:C0603
- removed PWR_IN: 5566-2, con-molex:5566-2
- removed TME1205S: (no value), dc-dc-converter:NME
- moved L1 132.7 mm to (79.8, 81.5)
- moved C1 130.8 mm to (86.4, 79.2), turned to 90 degrees
- moved PWR_IN1 128.8 mm to (64.3, 81.3), turned to 180 degrees
- moved C2 124.9 mm to (72.9, 78.7), turned to 270 degrees
- moved R-78-1.0 101.2 mm to (79.0, 55.9), turned to 180 degrees
Connections:
- removed net N$36: C2.1, L1.1, PWR_IN1.1
- net 5V: no longer C5.1, TME1205S.4
- net GND: no longer C4.2, C5.2, PWR_IN.2, TME1205S.1, TME1205S.3
- net VCC: now also C2.1, L1.1, PWR_IN1.1; no longer C4.1, PWR_IN.1, TME1205S.2
Routing:
- net N$16: track 0.00 -> 27.4 mm, vias 0 -> 1
- net VCC: track 199.9 -> 175.7 mm, vias 2 -> 3
- net 5V: track 181.3 -> 188.1 mm, vias 2 -> 4

Commit message: Mainboard fixes
Parts:
- removed R-78-1.0: (no value), v-reg:78XXS
- added PS1: R-785.0-1.0, R-785.0-1.0:CONV_R-785.0-1.0
- moved U1 2.29 mm to (69.8, 52.3)
Connections:
- removed net GND2: U2.26
- removed net GND3: U2.20
- net 5V: now also PS1.3; no longer R-78-1.0.OUT
- net GND: now also PS1.2, U2.20, U2.26; no longer R-78-1.0.GND
- net N$16: now also PS1.1; no longer R-78-1.0.IN
Routing:
- net GND: track 74.8 -> 154.1 mm, vias 7 -> 13
- net 5V: track 188.1 -> 209.9 mm
- net 3V3: track 83.9 -> 79.3 mm
- net N$16: track 27.4 -> 30.0 mm
- net CTX: track 16.9 -> 14.8 mm
- net CRX: track 15.6 -> 14.5 mm
- net CANL: track 9.67 -> 9.07 mm

Commit message: BMS V3 hardware
Parts:
- removed C2: 10μF, rcl:C0603
- removed C6: 0.1μF, rcl:C0603
- removed CAN: 5566-2, con-molex:5566-2
- removed CTSREF2: 1uf, rcl:C0603
- removed L1: 5.6 uH, inductor-neosid:SD8
- removed TEMPH: 5566-16, con-molex:5566-16
- removed TEMPR10, TEMPR11, TEMPR12, TEMPR13, TEMPR14, TEMPR15, TEMPR16, TEMPR9: 10k, rcl:R0603
- added C3, C4: 0.1μF, rcl:C0603
- added CAN1, CAN2, CAN3: 5566-2, con-molex:5566-2
- added R10, R19: 120, rcl:R0603
- added U3, U4, U5: CAN_TRANSCAN_TRANS, NFR23_v1.1:MAX3051ESA+
- C1: value 2.2μF -> 0.1μF
- CCOMHN, CCOMHP, CCOMLN, CCOMLP: device rcl:C0603 -> rcl:C050-035X075
- PS1: value R-785.0-1.0 -> TSR_1-2450; device R-785.0-1.0:CONV_R-785.0-1.0 -> dcdc_5v:TSR1-SINGLE_TRP
- U1: value MCP2562-E/SN -> CAN_TRANSCAN_TRANS; device MCP2562-E_SN:SOIC127P600X175-8N -> NFR23_v1.1:MAX3051ESA+
- moved C1 49.1 mm to (83.3, 30.2)
- moved R8 13.2 mm to (86.9, 47.2)
- moved U1 12.2 mm to (80.8, 47.0)
- moved C7 7.79 mm to (73.9, 53.3)
- moved COML 5.61 mm to (54.9, 5.33)
- moved R2 5.61 mm to (46.7, 9.14)
- moved RCOMHN 3.81 mm to (79.2, 1.65)
- moved CCOMHNG 3.56 mm to (76.2, 1.65)
- moved PS1 3.06 mm to (70.9, 61.5)
- moved CNPN1-1 2.34 mm to (89.4, 17.5), turned to 0 degrees
- moved CCOMHN 1.70 mm to (84.1, 2.16)
- moved COMH 1.05 mm to (90.4, 6.73)
- moved ESDCOML 1.05 mm to (68.8, 4.32)
- moved CCOMLP 0.76 mm to (65.3, 5.84)
- moved CCOMLN 0.51 mm to (65.3, 2.03)
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Connections:
- removed net CANH: CAN.1, R8.1, U1.7
- removed net CANL: CAN.2, R8.2, U1.6
- removed net CRX: U$3.30-CRX3, U1.4
- removed net CS0: U$3.38-A14/CS/IN1
- removed net CSTBY: U$3.29-TX7, U1.8
- removed net CTX: U$3.31-CTX3, U1.1
- removed net MISO: U$3.12-MISO/MQSL
- removed net MOSI: U$3.11-MOSI/CTX1
- removed net N$16: C1.1, L1.2, PS1.1
- removed net N$30: R17.1, U2.29
- removed net SCK: U$3.13-SCK/LED
- removed net SPI_RDY: U$3.17-A3/TX4/SDA1
- removed net TEMP12: IC2.58, TEMPH.4, TEMPR12.2
- removed net TSREF-1: CTSREF2.2, IC2.51, TEMPR10.1, TEMPR11.1, TEMPR12.1, TEMPR13.1, TEMPR14.1, TEMPR15.1, TEMPR16.1, TEMPR9.1
- new net CANH1: CAN1.1, R10.1, U5.7
- new net CANH2: CAN2.1, R8.1, U1.7
- new net CANH3: CAN3.1, R19.1, U3.7, U4.7
- new net CANL1: CAN1.2, R10.2, U5.6
- new net CANL2: CAN2.2, R8.2, U1.6
- new net CANL3: CAN3.2, R19.2, U3.6, U4.6
- new net CRX1: U$3.23-A9/CRX1/MCLK1, U5.4
- new net CRX2: U$3.0-RX1/CS1/CRX2, U1.4
- new net CRX3: U$3.30-CRX3, U3.4
- new net CTX1: U$3.22-A8/CTX1, U5.1
- new net CTX2: U$3.1-TX1/MISO1/CTX2, U1.1
- new net CTX3: U$3.31-CTX3, U3.1
- new net ESPCANRX: U2.32, U4.4
- new net ESPCANTX: U2.29, U4.1
- new net N$11: R17.1, U2.22
- new net N$41: IC2.51
- net 3V3: now also C1.2, C3.2, C4.2, C7.2, U1.3, U3.3, U4.3, U5.3; no longer C7.1, U1.5
- net 5V: no longer C6.1, U1.3
- net CONTACTORN_CTRL: now also U$3.10-CS\MQSR; no longer U$3.22-A8/CTX1
- net COOLANT_CTRL: now also U$3.11-MOSI/CTX1; no longer U$3.23-A9/CRX1/MCLK1
- net GND: now also C1.1, C3.1, C4.1, C7.1, U1.8, U3.2, U3.8, U4.2, U4.8, U5.2, U5.8; no longer C1.2, C2.2, C6.2, C7.2, CTSREF2.1, TEMPH.10, TEMPH.11, TEMPH.12, TEMPH.13, TEMPH.14, TEMPH.15, TEMPH.16, TEMPH.9
- net NFAULT: now also IC2.62
- net RX_ESP: now also U$3.29-TX7; no longer U$3.1-TX1/MISO1/CTX2
- net TEMP10: no longer TEMPH.2, TEMPR10.2
- net TEMP11: no longer TEMPH.3, TEMPR11.2
- net TEMP13: no longer TEMPH.5, TEMPR13.2
- net TEMP14: no longer TEMPH.6, TEMPR14.2
- net TEMP15: no longer TEMPH.7, TEMPR15.2
- net TEMP16: no longer TEMPH.8, TEMPR16.2
- net TEMP9: no longer TEMPH.1, TEMPR9.2
- net TX_ESP: now also U$3.28-RX7; no longer U$3.0-RX1/CS1/CRX2
- net VCC: now also PS1.1; no longer C2.1, L1.1
Routing:
- net NFAULT: track 0.00 -> 94.0 mm, vias 0 -> 1
- net CRX1: track 0.00 -> 85.6 mm, vias 0 -> 2
- net CRX2: track 0.00 -> 83.1 mm, vias 0 -> 4
- net CTX2: track 0.00 -> 81.0 mm, vias 0 -> 4
- net ESPCANRX: track 0.00 -> 79.2 mm, vias 0 -> 1
- net CTX1: track 0.00 -> 78.3 mm, vias 0 -> 2
- net ESPCANTX: track 0.00 -> 65.7 mm, vias 0 -> 1
- net TEMP9: track 46.9 -> 0.00 mm
- net TEMP10: track 44.3 -> 0.00 mm, vias 2 -> 0
- net TSREF-1: track 42.3 -> 0.00 mm, vias 2 -> 0
- net COOLANT_CTRL: track 15.0 -> 55.5 mm, vias 0 -> 2
- net TEMP11: track 34.9 -> 0.00 mm, vias 2 -> 0
- net CRX3: track 0.00 -> 33.7 mm, vias 0 -> 2
- net 5V: track 209.9 -> 176.9 mm, vias 4 -> 2
- net TEMP12: track 31.4 -> 0.00 mm, vias 2 -> 0
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Other:
- board text added: "BMS Main Board V3"
- board text added: "GPIO"
- board text added: "Joshua Feist, Lance Go, Luc Ah-Hot, Isaac Kim Jan 2023"
- board text removed: "BMS Main Board V1.1"
- board text removed: "COMH"
- board text removed: "COML"
- board text removed: "DIEEEEEE!!!!!!"
- board text removed: "Luc Ah-Hot, Joshua Feist, Lance Go, Isaac Kim Jan 2022"
