File: Hardware/Main controller 79656/esp_teensy_bridge.sch (EAGLE design)
At the start: 93 parts, among them IC2 PBQ79656PAPTQ1, Q5 VISHAY_SIS862DN-T1-GE3VISHAY_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, Q6 VISHAY_SIS862DN-T1-GE3VISHAY_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, Q7 VISHAY_SIS862DN-T1-GE3VISHAY_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, Q8 VISHAY_SIS862DN-T1-GE3VISHAY_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, T2 PBHV8115X, 115, U1 CAN_TRANSCAN_TRANS, U2 ESP32-DEVKITC-32D, U3 CAN_TRANSCAN_TRANS, U4 CAN_TRANSCAN_TRANS, U5 CAN_TRANSCAN_TRANS, X1 5566-12

Commit message: Mainboard update (#101)
* Switched to eGaN FETs

* Switched to single connector for mainboard, generated gerbers

* Labelled HV/LV on mainboard

* Updates from feedback

* Changes, gerbers
Parts:
- removed CAN1, CAN2, CAN3, COMH, COML, CONTACTOR_N, CONTACTOR_P, CONTACTOR_PRECHARGE, COOLANT, PWR_IN1: 5566-2, con-molex:5566-2
- removed Q5, Q6, Q7, Q8: VISHAY_SIS862DN-T1-GE3VISHAY_SIS862DN-T1-GE3_0_0, Vishay - SIS862DN-T1-GE3:VISHAY_SIS862DN-T1-GE3VISHAY_SIS862DN-T1-GE3_0_0
- removed X1: 5566-12, con-molex:5566-12
- added CFET1, CFET2, CFET3, CFET4, CVCC: 10uf, rcl:C-EUC0805
- added J1, J2: DF11-4DP-2DSA(24), hirose_connectors:DF11-4DP-2DSA(24)
- added J3: TE_AMP_SURESEAL_26, TE_Sureseal:TE_AMP_SURESEAL_26
- added Q1, Q2, Q3, Q4: EPC2065, EPCGaNFET:EPC2065
- added R20, R21, R22, R23: 300, rcl:R-US_R0603
- added R24: 6k, rcl:R-US_R0603
- added R25, R26: 1k, rcl:R-US_R0603
- CCOMHN, CCOMHP, CCOMLN, CCOMLP: device rcl:C-EU050-035X075 -> rcl:C-EU075-032X103
Connections:
- removed net N$12: CONTACTOR_P-2.S, Q7.D
- removed net N$14: U$3.14-A0/TX3/SPDIF_OUT, X1-1.S
- removed net N$17: U$3.15-A1/RX3/SPDIF_IN, X1-2.S
- removed net N$18: U$3.18-A4/SDA0, X1-3.S
- removed net N$19: U$3.19-A5/SCL0, X1-4.S
- removed net N$20: U$3.24-A10/TX6/SCL2, X1-5.S
- removed net N$21: U$3.25-A11/RX6/SDA2, X1-6.S
- removed net N$22: U$3.40-A16/CS1, X1-7.S
- removed net N$23: U$3.32-OUT1B, X1-8.S
- removed net N$24: U$3.9-OUT1C, X1-9.S
- removed net N$25: U$3.6-OUT1D, X1-10.S
- removed net N$26: U$3.33-MCLK2, X1-12.S
- removed net N$27: U$3.2-OUT2, X1-11.S
- removed net N$5: COOLANT-2.S, Q5.D
- removed net N$6: CONTACTOR_PRECHARGE-2.S, Q8.D
- new net CONTACTORN_OUT: J3.24, Q3.3, Q3.5, Q3.7, R13.1
- new net CONTACTORPRECHARGE_OUT: J3.26, Q1.3, Q1.5, Q1.7, R11.1
- new net CONTACTORP_OUT: J3.25, Q2.3, Q2.5, Q2.7, R12.1
- new net COOLING_OUT: J3.17, J3.18, J3.19, Q4.3, Q4.5, Q4.7, R14.1
- new net N$15: Q1.1, R20.1
- new net N$16: Q2.1, R21.1
- new net N$30: Q3.1, R23.1
- new net N$36: Q4.1, R22.1
- new net NFAULT_3V3: U$1.A3, U$3.16-A2/RX4/SCL1
- new net SHUTDOWN_IN: J3.11, R24.2, R26.1
- new net SHUTDOWN_SIGNAL: R24.1, R25.2, U$3.38-A14/CS/IN1
- net CANH1: now also J3.4; no longer CAN1-1.S
- net CANH2: now also J3.3; no longer CAN2-1.S
- net CANH3: now also J3.2; no longer CAN3-1.S
- net CANL1: now also J3.10; no longer CAN1-2.S
- net CANL2: now also J3.9; no longer CAN2-2.S
- net CANL3: now also J3.8; no longer CAN3-2.S
- net COMHN: now also J1.4; no longer COMH-1.S
- net COMHP: now also J1.3; no longer COMH-2.S
- net COMLN: now also J2.1; no longer COML-1.S
- net COMLP: now also J2.2; no longer COML-2.S
- net CONTACTORN_CTRL: now also R23.2; no longer Q6.G, R13.1
- net CONTACTORPRECHARGE_CTRL: now also R20.2; no longer Q8.G, R11.1
- net CONTACTORP_CTRL: now also R21.2; no longer Q7.G, R12.1
- net COOLANT_CTRL: now also R22.2; no longer Q5.G, R14.1
- net GND: now also CFET1.2, CFET2.1, CFET3.1, CFET4.1, CVCC.1, J3.12, J3.13, J3.5, J3.6, J3.7, Q1.2, Q1.4, Q1.6, Q1.8, Q2.2, Q2.4, Q2.6, Q2.8, Q3.2, Q3.4, Q3.6, Q3.8, Q4.2, Q4.4, Q4.6, Q4.8, R25.1; no longer PWR_IN1-2.S, Q5.1_S, Q5.2_S, Q5.3_S, Q6.1_S, Q6.2_S, Q6.3_S, Q7.1_S, Q7.2_S, Q7.3_S, Q8.1_S, Q8.2_S, Q8.3_S
- net N$13: now also LED1.C, R11.2; no longer LED4.A, R14.2
- net N$130: now also CVCC.2
- net N$2: now also J3.14, R26.2; no longer CONTACTOR_N-2.S, Q6.D
- net N$3: now also LED4.C, R14.2; no longer LED1.A, R11.2
- net N$4: now also LED3.C, R13.2; no longer LED2.A, R12.2
- net N$9: now also LED2.C, R12.2; no longer LED3.A, R13.2
- net NFAULT: now also U$1.B3; no longer U$3.16-A2/RX4/SCL1
- net VCC: now also CFET1.1, CFET2.2, CFET3.2, CFET4.2, J3.1, LED1.A, LED2.A, LED3.A, LED4.A; no longer CONTACTOR_N-1.S, CONTACTOR_P-1.S, CONTACTOR_PRECHARGE-1.S, COOLANT-1.S, LED1.C, LED2.C, LED3.C, LED4.C, PWR_IN1-1.S
Other:
- moved on the sheet: LED1, LED2, LED3, LED4, R1, R5, R6, R7
