File: Hardware/Sense PCBs/sense_pcb_a.brd (EAGLE design)
At the start: 20 x 247 mm, 6 parts, among them J1 DF11-18DP-2DSA(24)

Commit message: sense pcb a
Parts:
- added U$10, U$6, U$7, U$8, U$9: BB_CONTACT, sense_pcb_components:BB_CONTACT
- added U$11: FUSE, sense_pcb_components:FUSE_PADS
- added U$12, U$13, U$14, U$15, U$16, U$17, U$18, U$19, U$20, U$21, U$22, U$23, U$24, U$25, U$26, U$27, U$28, U$29, U$30, U$31: THERM_PIN, sense_pcb_components:THERM_PIN
- moved J1 16.0 mm to (-9.53, 243.3), flipped to the bottom
- moved U$5 8.38 mm to (-1.40, 189.6), turned to 0 degrees
Connections:
- new net N$11: J1.3, J1.4, U$4.P$1, U$4.P$3, U$4.P$5
- new net N$2: U$1.P$2, U$1.P$4, U$1.P$6, U$6.P$1
- new net N$4: U$2.P$2, U$2.P$4, U$2.P$6, U$7.P$1
- new net N$5: U$10.P$1, U$5.P$2, U$5.P$4, U$5.P$6
- new net N$6: U$3.P$2, U$3.P$4, U$3.P$6, U$8.P$1
- new net N$8: U$4.P$2, U$4.P$4, U$4.P$6, U$9.P$1
- new net THERM1: J1.14, U$22.P$1, U$23.P$1
- new net THERM2: J1.15, U$24.P$1, U$25.P$1
- new net THERM3: J1.16, U$26.P$1, U$27.P$1
- new net THERM4: J1.17, U$28.P$1, U$29.P$1
- new net THERM5: J1.18, U$30.P$1, U$31.P$1
- new net THERMGND: J1.13, U$12.P$1, U$13.P$1, U$14.P$1, U$15.P$1, U$16.P$1, U$17.P$1, U$18.P$1, U$19.P$1, U$20.P$1, U$21.P$1
- net N$1: now also J1.11, J1.12, U$11.P$1, U$11.P$3, U$11.P$5; no longer J1.1, J1.2, U$1.P$1, U$1.P$3, U$1.P$5
- net N$3: now also J1.1, J1.2, U$5.P$1, U$5.P$3, U$5.P$5; no longer J1.3, J1.4, U$2.P$1, U$2.P$3, U$2.P$5
- net N$7: now also J1.10, J1.9, U$1.P$1, U$1.P$3, U$1.P$5; no longer J1.7, J1.8, U$4.P$1, U$4.P$3, U$4.P$5
- net N$9: now also J1.7, J1.8, U$2.P$1, U$2.P$3, U$2.P$5; no longer J1.10, J1.9, U$5.P$1, U$5.P$3, U$5.P$5
Routing:
- net N$7: track 123.0 -> 364.9 mm
- net THERM5: track 0.00 -> 240.5 mm
- net THERMGND: track 0.00 -> 238.3 mm
- net THERM4: track 0.00 -> 197.6 mm
- net N$9: track 100.0 -> 285.2 mm
- net N$3: track 287.9 -> 120.2 mm
- net THERM3: track 0.00 -> 156.4 mm
- net N$11: track 0.00 -> 124.8 mm
- net N$1: track 367.8 -> 485.8 mm
- net THERM2: track 0.00 -> 116.3 mm
- net THERM1: track 0.00 -> 83.9 mm
- net N$6: track 0.00 -> 23.0 mm
- net N$8: track 0.00 -> 23.0 mm
- net N$2: track 0.00 -> 22.7 mm
- net N$5: track 0.00 -> 13.7 mm
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
Commit message: Äll sense boards done
Other:
- board text added: "THERM1"
- board text added: "THERM2"
- board text added: "THERM3"
- board text added: "THERM4"
- board text added: "THERM5"
Changed lines of the file:
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@@
 <wire x1="-2.8" y1="98.2" x2="0" y2="98.2" width="0.001" layer="20"/>
 <wire x1="0" y1="95.4" x2="-2.8" y2="98.2" width="0.001" layer="20"/>
+<text x="4.6482" y="201.7776" size="0.508" layer="21" font="vector" rot="R90">THERM1</text>
+<text x="4.6482" y="162.7632" size="0.508" layer="21" font="vector" rot="R90">THERM1</text>
+<text x="4.6482" y="147.1676" size="0.508" layer="21" font="vector" rot="R90">THERM2</text>
+<text x="4.572" y="122.6312" size="0.508" layer="21" font="vector" rot="R90">THERM2</text>
+<text x="4.3942" y="107.8738" size="0.508" layer="21" font="vector" rot="R90">THERM3</text>
+<text x="4.572" y="85.3694" size="0.508" layer="21" font="vector" rot="R90">THERM3</text>
+<text x="4.2164" y="63.2714" size="0.508" layer="21" font="vector" rot="R90">THERM4</text>
+<text x="4.4196" y="41.9862" size="0.508" layer="21" font="vector" rot="R90">THERM4</text>
+<text x="4.2926" y="21.7424" size="0.508" layer="21" font="vector" rot="R90">THERM5</text>
+<text x="4.445" y="8.4328" size="0.508" layer="21" rot="R90">THERM5</text>
 </plain>
 <attributes>
@@
 <contactref element="U$22" pad="P$1"/>
 <contactref element="U$23" pad="P$1"/>
-<contactref element="U$23" pad="P$1"/>
 <wire x1="2.4638" y1="245.3132" x2="3.5306" y2="244.2464" width="0.127" layer="1"/>
 <wire x1="3.683" y1="204.62510625" x2="3.683" y2="203.19729375" width="0.127" layer="1"/>
@@
 <contactref element="J1" pad="15"/>
 <contactref element="U$24" pad="P$1"/>
-<contactref element="U$25" pad="P$1"/>
 <contactref element="U$25" pad="P$1"/>
 <wire x1="4.4704" y1="243.3066" x2="4.4704" y2="242.7478" width="0.127" layer="1"/>
@@
 <contactref element="J1" pad="16"/>
 <contactref element="U$26" pad="P$1"/>
-<contactref element="U$27" pad="P$1"/>
 <contactref element="U$27" pad="P$1"/>
 <wire x1="4.4704" y1="245.3132" x2="4.4704" y2="244.4740375" width="0.127" layer="1"/>
@@
 <contactref element="U$28" pad="P$1"/>
 <contactref element="U$29" pad="P$1"/>
-<contactref element="U$29" pad="P$1"/>
 <wire x1="6.477" y1="243.3066" x2="6.477" y2="242.3377875" width="0.127" layer="1"/>
 <wire x1="6.477" y1="242.3377875" x2="4.2926" y2="240.1533875" width="0.127" layer="1"/>
@@
 <contactref element="J1" pad="18"/>
 <contactref element="U$30" pad="P$1"/>
-<contactref element="U$31" pad="P$1"/>
 <contactref element="U$31" pad="P$1"/>
 <wire x1="6.477" y1="245.3132" x2="6.477" y2="244.4740375" width="0.127" layer="1"/>
@@
 <contactref element="U$12" pad="P$1"/>
 <contactref element="U$13" pad="P$1"/>
-<contactref element="U$13" pad="P$1"/>
 <contactref element="U$14" pad="P$1"/>

Commit message: fixed outline, updated gerbers
Parts:
- U$11: value FUSE -> BB_CONTACT; device sense_pcb_components:FUSE_PADS -> sense_pcb_components:BB_CONTACT
- moved U$11 0.51 mm to (2.54, 2.03), turned to 0 degrees
Connections:
- net N$1: no longer U$11.P$3, U$11.P$5
Routing:
- net N$4: track 0.00 -> 23.1 mm
- net N$9: track 285.2 -> 285.8 mm
- net N$7: track 364.9 -> 365.5 mm
- net N$2: track 22.7 -> 23.2 mm
Other:
- board text added: "A"
