File: Hardware/Sense PCBs/sense_pcb_a.sch (EAGLE design)
At the start: 6 parts, among them J1 DF11-18DP-2DSA(24)

Commit message: sense pcb a
Parts:
- added U$10, U$6, U$7, U$8, U$9: BB_CONTACT, sense_pcb_components:BB_CONTACT
- added U$11: FUSE, sense_pcb_components:FUSE
- added U$12, U$13, U$14, U$15, U$16, U$17, U$18, U$19, U$20, U$21, U$22, U$23, U$24, U$25, U$26, U$27, U$28, U$29, U$30, U$31: THERM_PIN, sense_pcb_components:THERM_PIN
Connections:
- new net N$11: J1.3, J1.4, U$4.P$1
- new net N$2: U$1.P$2, U$6.P$1
- new net N$4: U$2.P$2, U$7.P$1
- new net N$5: U$10.P$1, U$5.P$2
- new net N$6: U$3.P$2, U$8.P$1
- new net N$8: U$4.P$2, U$9.P$1
- new net THERM1: J1.14, U$22.P$1, U$23.P$1
- new net THERM2: J1.15, U$24.P$1, U$25.P$1
- new net THERM3: J1.16, U$26.P$1, U$27.P$1
- new net THERM4: J1.17, U$28.P$1, U$29.P$1
- new net THERM5: J1.18, U$30.P$1, U$31.P$1
- new net THERMGND: J1.13, U$12.P$1, U$13.P$1, U$14.P$1, U$15.P$1, U$16.P$1, U$17.P$1, U$18.P$1, U$19.P$1, U$20.P$1, U$21.P$1
- net N$1: now also J1.11, J1.12, U$11.P$1; no longer J1.1, J1.2, U$1.P$1
- net N$3: now also J1.1, J1.2, U$5.P$1; no longer J1.3, J1.4, U$2.P$1
- net N$7: now also J1.10, J1.9, U$1.P$1; no longer J1.7, J1.8, U$4.P$1
- net N$9: now also J1.7, J1.8, U$2.P$1; no longer J1.10, J1.9, U$5.P$1

Commit message: fixed outline, updated gerbers
Parts:
- U$11: value FUSE -> BB_CONTACT; device sense_pcb_components:FUSE -> sense_pcb_components:BB_CONTACT
Changed lines of the file:
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@@
 <part name="U$9" library="sense_pcb_components" deviceset="BB_CONTACT" device=""/>
 <part name="U$10" library="sense_pcb_components" deviceset="BB_CONTACT" device=""/>
-<part name="U$11" library="sense_pcb_components" deviceset="FUSE" device=""/>
 <part name="U$12" library="sense_pcb_components" deviceset="THERM_PIN" device=""/>
 <part name="U$13" library="sense_pcb_components" deviceset="THERM_PIN" device=""/>
@@
 <part name="U$30" library="sense_pcb_components" deviceset="THERM_PIN" device=""/>
 <part name="U$31" library="sense_pcb_components" deviceset="THERM_PIN" device=""/>
+<part name="U$11" library="sense_pcb_components" deviceset="BB_CONTACT" device=""/>
 </parts>
 <sheets>
@@
 <instance part="U$9" gate="G$1" x="27.94" y="10.16" smashed="yes" rot="R270"/>
 <instance part="U$10" gate="G$1" x="35.56" y="10.16" smashed="yes" rot="R270"/>
-<instance part="U$11" gate="G$1" x="-5.08" y="7.62" smashed="yes" rot="R90"/>
 <instance part="U$12" gate="G$1" x="22.86" y="83.82" smashed="yes" rot="R270"/>
 <instance part="U$13" gate="G$1" x="22.86" y="83.82" smashed="yes" rot="R270"/>
@@
 <instance part="U$30" gate="G$1" x="35.56" y="83.82" smashed="yes" rot="R270"/>
 <instance part="U$31" gate="G$1" x="35.56" y="83.82" smashed="yes" rot="R270"/>
+<instance part="U$11" gate="G$1" x="-5.08" y="15.24" smashed="yes" rot="R270"/>
 </instances>
 <busses>
@@
 <net name="N$1" class="0">
 <segment>
-<pinref part="U$11" gate="G$1" pin="P$1"/>
-<wire x1="-5.08" y1="17.78" x2="-5.08" y2="43.18" width="0.1524" layer="91"/>
+<wire x1="-5.08" y1="15.24" x2="-5.08" y2="43.18" width="0.1524" layer="91"/>
 <wire x1="-5.08" y1="43.18" x2="17.78" y2="43.18" width="0.1524" layer="91"/>
 <pinref part="J1" gate="A" pin="11"/>
@@
 <wire x1="17.78" y1="78.74" x2="20.32" y2="78.74" width="0.1524" layer="91"/>
 <junction x="17.78" y="78.74"/>
+<pinref part="U$11" gate="G$1" pin="P$1"/>
 </segment>
 </net>
